File: UTS Mini Mixing Desk - Compressor.kicad_sch (KiCad schematic)
At the start: 0 parts

Commit message: add Docs & fix name & all the other shit
Other:
- note added: "UTS Mini Mixing Desk - Compressor - one sheet per section"
- note removed: "Steer 500 compressor - one sheet per section"
- company: 500-series module -> UTS Mini Mixing Desk
- title: Steer 500 Compressor -> UTS Mini Mixing Desk - Compressor
Changed lines of the file:
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@@
 	(generator "eeschema")
 	(generator_version "9.0")
-	(paper "A3")
+	(paper "A4")
 	(title_block
-		(title "Steer 500 Compressor")
+		(title "UTS Mini Mixing Desk - Compressor")
 		(date "2026-08-31")
 		(rev "A")
-		(company "500-series module")
-	)
-	(text "Steer 500 compressor - one sheet per section"
-		(exclude_from_sim no)
-		(at 30 25 0)
+		(company "UTS Mini Mixing Desk")
+	)
+	(text "UTS Mini Mixing Desk - Compressor - one sheet per section"
+		(exclude_from_sim no)
+		(at 49.53 49.77 0)
 		(effects
 			(font
@@
 	)
 	(sheet
-		(at 182.4 40)
-		(size 44.45 25.4)
-		(exclude_from_sim no)
-		(in_bom yes)
-		(on_board yes)
-		(dnp no)
+		(at 201.93 64.77)
+		(size 44.45 25.4)
+		(exclude_from_sim no)
+		(in_bom yes)
+		(on_board yes)
+		(dnp no)
+		(fields_autoplaced yes)
 		(stroke
 			(width 0.1524)
@@
 		)
 		(property "Sheetname" "3 VCA"
-			(at 182.4 39.3 0)
+			(at 201.93 64.0584 0)
 			(effects
 				(font
@@
 		)
 		(property "Sheetfile" "vca.kicad_sch"
-			(at 182.4 66.1 0)
-			(effects
-				(font
-					(size 1.27 1.27)
-				)
-				(justify left top)
-			)
-		)
-		(instances
-			(project "steer500-sections"
+			(at 201.93 90.7546 0)
+			(effects
+				(font
+					(size 1.27 1.27)
+				)
+				(justify left top)
+			)
+		)
+		(instances
+			(project "UTS Mini Mixing Desk - Compressor"
 				(path "/fdeae63a-37f5-58fb-b342-cb68d8a6bfbc"
 					(page "4")
@@
 	)
 	(sheet
-		(at 30 90.8)
-		(size 44.45 25.4)
-		(exclude_from_sim no)
-		(in_bom yes)
-		(on_board yes)
-		(dnp no)
+		(at 49.53 115.57)
+		(size 44.45 25.4)
+		(exclude_from_sim no)
+		(in_bom yes)
+		(on_board yes)
+		(dnp no)
+		(fields_autoplaced yes)
 		(stroke
 			(width 0.1524)
@@
 		)
 		(property "Sheetname" "4 Output"
-			(at 30 90.1 0)
+			(at 49.53 114.8584 0)
 			(effects
 				(font
@@
 		)
 		(property "Sheetfile" "output.kicad_sch"
-			(at 30 116.9 0)
-			(effects
-				(font
-					(size 1.27 1.27)
-				)
-				(justify left top)
-			)
-		)
-		(instances
-			(project "steer500-sections"
+			(at 49.53 141.5546 0)
+			(effects
+				(font
+					(size 1.27 1.27)
+				)
+				(justify left top)
+			)
+		)
+		(instances
+			(project "UTS Mini Mixing Desk - Compressor"
 				(path "/fdeae63a-37f5-58fb-b342-cb68d8a6bfbc"
 					(page "5")
@@
 	)
 	(sheet
-		(at 106.2 40)
-		(size 44.45 25.4)
-		(exclude_from_sim no)
-		(in_bom yes)
-		(on_board yes)
-		(dnp no)
+		(at 125.73 64.77)
+		(size 44.45 25.4)
+		(exclude_from_sim no)
+		(in_bom yes)
+		(on_board yes)
+		(dnp no)
+		(fields_autoplaced yes)
 		(stroke
 			(width 0.1524)
@@
 		)
 		(property "Sheetname" "2 Input"
-			(at 106.2 39.3 0)
+			(at 125.73 64.0584 0)
 			(effects
 				(font
@@
 		)
 		(property "Sheetfile" "input.kicad_sch"
-			(at 106.2 66.1 0)
-			(effects
-				(font
-					(size 1.27 1.27)
-				)
-				(justify left top)
-			)
-		)
-		(instances
-			(project "steer500-sections"
+			(at 125.73 90.7546 0)
+			(effects
+				(font
+					(size 1.27 1.27)
+				)
+				(justify left top)
+			)
+		)
+		(instances
+			(project "UTS Mini Mixing Desk - Compressor"
 				(path "/fdeae63a-37f5-58fb-b342-cb68d8a6bfbc"
 					(page "3")
@@
 	)
 	(sheet
-		(at 106.2 90.8)
-		(size 44.45 25.4)
-		(exclude_from_sim no)
-		(in_bom yes)
-		(on_board yes)
-		(dnp no)
+		(at 125.73 115.57)
+		(size 44.45 25.4)
+		(exclude_from_sim no)
+		(in_bom yes)
+		(on_board yes)
+		(dnp no)
+		(fields_autoplaced yes)
 		(stroke
 			(width 0.1524)
@@
 		)
 		(property "Sheetname" "5 Sidechain"
-			(at 106.2 90.1 0)
+			(at 125.73 114.8584 0)
 			(effects
 				(font
@@
 		)
 		(property "Sheetfile" "sidechain.kicad_sch"
-			(at 106.2 116.9 0)
-			(effects
-				(font
-					(size 1.27 1.27)
-				)
-				(justify left top)
-			)
-		)
-		(instances
-			(project "steer500-sections"
+			(at 125.73 141.5546 0)
+			(effects
+				(font
+					(size 1.27 1.27)
+				)
+				(justify left top)
+			)
+		)
+		(instances
+			(project "UTS Mini Mixing Desk - Compressor"
 				(path "/fdeae63a-37f5-58fb-b342-cb68d8a6bfbc"
 					(page "6")
@@
 	)
 	(sheet
-		(at 30 40)
-		(size 44.45 25.4)
-		(exclude_from_sim no)
-		(in_bom yes)
-		(on_board yes)
-		(dnp no)
+		(at 49.53 64.77)
+		(size 44.45 25.4)
+		(exclude_from_sim no)
+		(in_bom yes)
+		(on_board yes)
+		(dnp no)
+		(fields_autoplaced yes)
 		(stroke
 			(width 0.1524)
@@
 		)
 		(property "Sheetname" "1 Connector"
-			(at 30 39.3 0)
+			(at 49.53 64.0584 0)
 			(effects
 				(font
@@
 		)
 		(property "Sheetfile" "connector.kicad_sch"
-			(at 30 66.1 0)
-			(effects
-				(font
-					(size 1.27 1.27)
-				)
-				(justify left top)
-			)
-		)
-		(instances
-			(project "steer500-sections"
+			(at 49.53 90.7546 0)
+			(effects
+				(font
+					(size 1.27 1.27)
+				)
+				(justify left top)
+			)
+		)
+		(instances
+			(project "UTS Mini Mixing Desk - Compressor"
 				(path "/fdeae63a-37f5-58fb-b342-cb68d8a6bfbc"
 					(page "2")
@@
 	)
 	(sheet
-		(at 182.4 90.8)
-		(size 44.45 25.4)
-		(exclude_from_sim no)
-		(in_bom yes)
-		(on_board yes)
-		(dnp no)
+		(at 201.93 115.57)
+		(size 44.45 25.4)
+		(exclude_from_sim no)
+		(in_bom yes)
+		(on_board yes)
+		(dnp no)
+		(fields_autoplaced yes)
 		(stroke
 			(width 0.1524)
@@
 		)
 		(property "Sheetname" "6 Power"
-			(at 182.4 90.1 0)
+			(at 201.93 114.8584 0)
 			(effects
 				(font
@@
 		)
 		(property "Sheetfile" "power.kicad_sch"
-			(at 182.4 116.9 0)
-			(effects
-				(font
-					(size 1.27 1.27)
-				)
-				(justify left top)
-			)
-		)
-		(instances
-			(project "steer500-sections"
+			(at 201.93 141.5546 0)
+			(effects
+				(font
+					(size 1.27 1.27)
+				)
+				(justify left top)
+			)
+		)
+		(instances
+			(project "UTS Mini Mixing Desk - Compressor"
 				(path "/fdeae63a-37f5-58fb-b342-cb68d8a6bfbc"
 					(page "7")
