File: connector.kicad_sch (KiCad schematic)
At the start: 1 part, among them J1 500 card edge

Commit message: add Docs & fix name & all the other shit
Other:
- company: Steer 500 -> UTS Mini Mixing Desk
- title: Steer 500 - 1 Connector -> UTS Mini Mixing Desk - Compressor
Changed lines of the file:
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@@
 	(paper "User" 200 150)
 	(title_block
-		(title "Steer 500 - 1 Connector")
+		(title "UTS Mini Mixing Desk - Compressor")
 		(date "2026-08-31")
 		(rev "A")
-		(company "Steer 500")
+		(company "UTS Mini Mixing Desk")
 	)
 	(no_connect
@@
 		)
 		(instances
-			(project "steer500-sections"
+			(project "UTS Mini Mixing Desk - Compressor"
 				(path "/fdeae63a-37f5-58fb-b342-cb68d8a6bfbc/a71beffb-08c5-50af-b047-4c3106cc907a"
 					(reference "#PWRCO000")
@@
 		)
 		(instances
-			(project "steer500-sections"
+			(project "UTS Mini Mixing Desk - Compressor"
 				(path "/fdeae63a-37f5-58fb-b342-cb68d8a6bfbc/a71beffb-08c5-50af-b047-4c3106cc907a"
 					(reference "#PWRCO001")
@@
 		)
 		(instances
-			(project "steer500-sections"
+			(project "UTS Mini Mixing Desk - Compressor"
 				(path "/fdeae63a-37f5-58fb-b342-cb68d8a6bfbc/a71beffb-08c5-50af-b047-4c3106cc907a"
 					(reference "#PWRCO002")
@@
 		)
 		(instances
-			(project "steer500-sections"
+			(project "UTS Mini Mixing Desk - Compressor"
 				(path "/fdeae63a-37f5-58fb-b342-cb68d8a6bfbc/a71beffb-08c5-50af-b047-4c3106cc907a"
 					(reference "J1")
