File: input.kicad_sch (KiCad schematic)
At the start: 14 parts, among them U1 NE5532

Commit message: add Docs & fix name & all the other shit
Parts:
- R8: value 47R -> 75R
Other:
- company: Steer 500 -> UTS Mini Mixing Desk
- title: Steer 500 - 2 Input -> UTS Mini Mixing Desk - Compressor
Changed lines of the file:
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@@
 	(paper "User" 269.24 150)
 	(title_block
-		(title "Steer 500 - 2 Input")
+		(title "UTS Mini Mixing Desk - Compressor")
 		(date "2026-08-31")
 		(rev "A")
-		(company "Steer 500")
+		(company "UTS Mini Mixing Desk")
 	)
 	(junction
@@
 		)
 		(instances
-			(project "steer500-sections"
+			(project "UTS Mini Mixing Desk - Compressor"
 				(path "/fdeae63a-37f5-58fb-b342-cb68d8a6bfbc/5797578f-278c-54d6-a28d-0cf0ddb33cbf"
 					(reference "#PWRIN002")
@@
 		)
 		(instances
-			(project "steer500-sections"
+			(project "UTS Mini Mixing Desk - Compressor"
 				(path "/fdeae63a-37f5-58fb-b342-cb68d8a6bfbc/5797578f-278c-54d6-a28d-0cf0ddb33cbf"
 					(reference "R2")
@@
 		)
 		(instances
-			(project "steer500-sections"
+			(project "UTS Mini Mixing Desk - Compressor"
 				(path "/fdeae63a-37f5-58fb-b342-cb68d8a6bfbc/5797578f-278c-54d6-a28d-0cf0ddb33cbf"
 					(reference "C3")
@@
 		)
 		(instances
-			(project "steer500-sections"
+			(project "UTS Mini Mixing Desk - Compressor"
 				(path "/fdeae63a-37f5-58fb-b342-cb68d8a6bfbc/5797578f-278c-54d6-a28d-0cf0ddb33cbf"
 					(reference "#PWRIN003")
@@
 		)
 		(instances
-			(project "steer500-sections"
+			(project "UTS Mini Mixing Desk - Compressor"
 				(path "/fdeae63a-37f5-58fb-b342-cb68d8a6bfbc/5797578f-278c-54d6-a28d-0cf0ddb33cbf"
 					(reference "C2")
@@
 		)
 		(instances
-			(project "steer500-sections"
+			(project "UTS Mini Mixing Desk - Compressor"
 				(path "/fdeae63a-37f5-58fb-b342-cb68d8a6bfbc/5797578f-278c-54d6-a28d-0cf0ddb33cbf"
 					(reference "R1")
@@
 		)
 		(instances
-			(project "steer500-sections"
+			(project "UTS Mini Mixing Desk - Compressor"
 				(path "/fdeae63a-37f5-58fb-b342-cb68d8a6bfbc/5797578f-278c-54d6-a28d-0cf0ddb33cbf"
 					(reference "C1")
@@
 		)
 		(instances
-			(project "steer500-sections"
+			(project "UTS Mini Mixing Desk - Compressor"
 				(path "/fdeae63a-37f5-58fb-b342-cb68d8a6bfbc/5797578f-278c-54d6-a28d-0cf0ddb33cbf"
 					(reference "R3")
@@
 		)
 		(instances
-			(project "steer500-sections"
+			(project "UTS Mini Mixing Desk - Compressor"
 				(path "/fdeae63a-37f5-58fb-b342-cb68d8a6bfbc/5797578f-278c-54d6-a28d-0cf0ddb33cbf"
 					(reference "C4")
@@
 		)
 		(instances
-			(project "steer500-sections"
+			(project "UTS Mini Mixing Desk - Compressor"
 				(path "/fdeae63a-37f5-58fb-b342-cb68d8a6bfbc/5797578f-278c-54d6-a28d-0cf0ddb33cbf"
 					(reference "#PWRIN001")
@@
 		)
 		(instances
-			(project "steer500-sections"
+			(project "UTS Mini Mixing Desk - Compressor"
 				(path "/fdeae63a-37f5-58fb-b342-cb68d8a6bfbc/5797578f-278c-54d6-a28d-0cf0ddb33cbf"
 					(reference "R5")
@@
 		)
 		(instances
-			(project "steer500-sections"
+			(project "UTS Mini Mixing Desk - Compressor"
 				(path "/fdeae63a-37f5-58fb-b342-cb68d8a6bfbc/5797578f-278c-54d6-a28d-0cf0ddb33cbf"
 					(reference "R7")
@@
 		)
 		(instances
-			(project "steer500-sections"
+			(project "UTS Mini Mixing Desk - Compressor"
 				(path "/fdeae63a-37f5-58fb-b342-cb68d8a6bfbc/5797578f-278c-54d6-a28d-0cf0ddb33cbf"
 					(reference "R6")
@@
 		)
 		(instances
-			(project "steer500-sections"
+			(project "UTS Mini Mixing Desk - Compressor"
 				(path "/fdeae63a-37f5-58fb-b342-cb68d8a6bfbc/5797578f-278c-54d6-a28d-0cf0ddb33cbf"
 					(reference "U1")
@@
 		)
 		(instances
-			(project "steer500-sections"
+			(project "UTS Mini Mixing Desk - Compressor"
 				(path "/fdeae63a-37f5-58fb-b342-cb68d8a6bfbc/5797578f-278c-54d6-a28d-0cf0ddb33cbf"
 					(reference "R4")
@@
 			)
 		)
-		(property "Value" "47R"
+		(property "Value" "75R"
 			(at 101.6 99.69 0)
 			(effects
@@
 		)
 		(instances
-			(project "steer500-sections"
+			(project "UTS Mini Mixing Desk - Compressor"
 				(path "/fdeae63a-37f5-58fb-b342-cb68d8a6bfbc/5797578f-278c-54d6-a28d-0cf0ddb33cbf"
 					(reference "R8")
@@
 		)
 		(instances
-			(project "steer500-sections"
+			(project "UTS Mini Mixing Desk - Compressor"
 				(path "/fdeae63a-37f5-58fb-b342-cb68d8a6bfbc/5797578f-278c-54d6-a28d-0cf0ddb33cbf"
 					(reference "RV1")
@@
 		)
 		(instances
-			(project "steer500-sections"
+			(project "UTS Mini Mixing Desk - Compressor"
 				(path "/fdeae63a-37f5-58fb-b342-cb68d8a6bfbc/5797578f-278c-54d6-a28d-0cf0ddb33cbf"
 					(reference "#PWRIN000")
