File: output.kicad_sch (KiCad schematic)
At the start: 17 parts, among them SW1 BYPASS, U2 NE5532, U5 NE5532

Commit message: add Docs & fix name & all the other shit
Other:
- company: Steer 500 -> UTS Mini Mixing Desk
- title: Steer 500 - 4 Output -> UTS Mini Mixing Desk - Compressor
Changed lines of the file:
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@@
 	(paper "User" 246.38 170.18)
 	(title_block
-		(title "Steer 500 - 4 Output")
+		(title "UTS Mini Mixing Desk - Compressor")
 		(date "2026-08-31")
 		(rev "A")
-		(company "Steer 500")
+		(company "UTS Mini Mixing Desk")
 	)
 	(junction
@@
 		)
 		(instances
-			(project "steer500-sections"
+			(project "UTS Mini Mixing Desk - Compressor"
 				(path "/fdeae63a-37f5-58fb-b342-cb68d8a6bfbc/3c12989f-7a47-57c9-9938-7ba13ccb2516"
 					(reference "#PWROU001")
@@
 		)
 		(instances
-			(project "steer500-sections"
+			(project "UTS Mini Mixing Desk - Compressor"
 				(path "/fdeae63a-37f5-58fb-b342-cb68d8a6bfbc/3c12989f-7a47-57c9-9938-7ba13ccb2516"
 					(reference "R83")
@@
 		)
 		(instances
-			(project "steer500-sections"
+			(project "UTS Mini Mixing Desk - Compressor"
 				(path "/fdeae63a-37f5-58fb-b342-cb68d8a6bfbc/3c12989f-7a47-57c9-9938-7ba13ccb2516"
 					(reference "R30")
@@
 		)
 		(instances
-			(project "steer500-sections"
+			(project "UTS Mini Mixing Desk - Compressor"
 				(path "/fdeae63a-37f5-58fb-b342-cb68d8a6bfbc/3c12989f-7a47-57c9-9938-7ba13ccb2516"
 					(reference "#PWROU000")
@@
 		)
 		(instances
-			(project "steer500-sections"
+			(project "UTS Mini Mixing Desk - Compressor"
 				(path "/fdeae63a-37f5-58fb-b342-cb68d8a6bfbc/3c12989f-7a47-57c9-9938-7ba13ccb2516"
 					(reference "#PWROU003")
@@
 		)
 		(instances
-			(project "steer500-sections"
+			(project "UTS Mini Mixing Desk - Compressor"
 				(path "/fdeae63a-37f5-58fb-b342-cb68d8a6bfbc/3c12989f-7a47-57c9-9938-7ba13ccb2516"
 					(reference "R28")
@@
 		)
 		(instances
-			(project "steer500-sections"
+			(project "UTS Mini Mixing Desk - Compressor"
 				(path "/fdeae63a-37f5-58fb-b342-cb68d8a6bfbc/3c12989f-7a47-57c9-9938-7ba13ccb2516"
 					(reference "SW1")
@@
 		)
 		(instances
-			(project "steer500-sections"
+			(project "UTS Mini Mixing Desk - Compressor"
 				(path "/fdeae63a-37f5-58fb-b342-cb68d8a6bfbc/3c12989f-7a47-57c9-9938-7ba13ccb2516"
 					(reference "C13")
@@
 		)
 		(instances
-			(project "steer500-sections"
+			(project "UTS Mini Mixing Desk - Compressor"
 				(path "/fdeae63a-37f5-58fb-b342-cb68d8a6bfbc/3c12989f-7a47-57c9-9938-7ba13ccb2516"
 					(reference "RV2")
@@
 		)
 		(instances
-			(project "steer500-sections"
+			(project "UTS Mini Mixing Desk - Compressor"
 				(path "/fdeae63a-37f5-58fb-b342-cb68d8a6bfbc/3c12989f-7a47-57c9-9938-7ba13ccb2516"
 					(reference "R26")
@@
 		)
 		(instances
-			(project "steer500-sections"
+			(project "UTS Mini Mixing Desk - Compressor"
 				(path "/fdeae63a-37f5-58fb-b342-cb68d8a6bfbc/3c12989f-7a47-57c9-9938-7ba13ccb2516"
 					(reference "U2")
@@
 		)
 		(instances
-			(project "steer500-sections"
+			(project "UTS Mini Mixing Desk - Compressor"
 				(path "/fdeae63a-37f5-58fb-b342-cb68d8a6bfbc/3c12989f-7a47-57c9-9938-7ba13ccb2516"
 					(reference "R29")
@@
 		)
 		(instances
-			(project "steer500-sections"
+			(project "UTS Mini Mixing Desk - Compressor"
 				(path "/fdeae63a-37f5-58fb-b342-cb68d8a6bfbc/3c12989f-7a47-57c9-9938-7ba13ccb2516"
 					(reference "R80")
@@
 		)
 		(instances
-			(project "steer500-sections"
+			(project "UTS Mini Mixing Desk - Compressor"
 				(path "/fdeae63a-37f5-58fb-b342-cb68d8a6bfbc/3c12989f-7a47-57c9-9938-7ba13ccb2516"
 					(reference "R34")
@@
 		)
 		(instances
-			(project "steer500-sections"
+			(project "UTS Mini Mixing Desk - Compressor"
 				(path "/fdeae63a-37f5-58fb-b342-cb68d8a6bfbc/3c12989f-7a47-57c9-9938-7ba13ccb2516"
 					(reference "U2")
@@
 		)
 		(instances
-			(project "steer500-sections"
+			(project "UTS Mini Mixing Desk - Compressor"
 				(path "/fdeae63a-37f5-58fb-b342-cb68d8a6bfbc/3c12989f-7a47-57c9-9938-7ba13ccb2516"
 					(reference "R33")
@@
 		)
 		(instances
-			(project "steer500-sections"
+			(project "UTS Mini Mixing Desk - Compressor"
 				(path "/fdeae63a-37f5-58fb-b342-cb68d8a6bfbc/3c12989f-7a47-57c9-9938-7ba13ccb2516"
 					(reference "R32")
@@
 		)
 		(instances
-			(project "steer500-sections"
+			(project "UTS Mini Mixing Desk - Compressor"
 				(path "/fdeae63a-37f5-58fb-b342-cb68d8a6bfbc/3c12989f-7a47-57c9-9938-7ba13ccb2516"
 					(reference "R82")
@@
 		)
 		(instances
-			(project "steer500-sections"
+			(project "UTS Mini Mixing Desk - Compressor"
 				(path "/fdeae63a-37f5-58fb-b342-cb68d8a6bfbc/3c12989f-7a47-57c9-9938-7ba13ccb2516"
 					(reference "R31")
@@
 		)
 		(instances
-			(project "steer500-sections"
+			(project "UTS Mini Mixing Desk - Compressor"
 				(path "/fdeae63a-37f5-58fb-b342-cb68d8a6bfbc/3c12989f-7a47-57c9-9938-7ba13ccb2516"
 					(reference "U5")
@@
 		)
 		(instances
-			(project "steer500-sections"
+			(project "UTS Mini Mixing Desk - Compressor"
 				(path "/fdeae63a-37f5-58fb-b342-cb68d8a6bfbc/3c12989f-7a47-57c9-9938-7ba13ccb2516"
 					(reference "SW1")
@@
 		)
 		(instances
-			(project "steer500-sections"
+			(project "UTS Mini Mixing Desk - Compressor"
 				(path "/fdeae63a-37f5-58fb-b342-cb68d8a6bfbc/3c12989f-7a47-57c9-9938-7ba13ccb2516"
 					(reference "U5")
@@
 		)
 		(instances
-			(project "steer500-sections"
+			(project "UTS Mini Mixing Desk - Compressor"
 				(path "/fdeae63a-37f5-58fb-b342-cb68d8a6bfbc/3c12989f-7a47-57c9-9938-7ba13ccb2516"
 					(reference "R81")
@@
 		)
 		(instances
-			(project "steer500-sections"
+			(project "UTS Mini Mixing Desk - Compressor"
 				(path "/fdeae63a-37f5-58fb-b342-cb68d8a6bfbc/3c12989f-7a47-57c9-9938-7ba13ccb2516"
 					(reference "#PWROU002")
