File: power.kicad_sch (KiCad schematic)
At the start: 44 parts, among them U1 NE5532, U2 NE5532, U3 NE5532, U4 NE5532, U5 NE5532, U6 NE5532

Commit message: add Docs & fix name & all the other shit
Other:
- company: Steer 500 -> UTS Mini Mixing Desk
- title: Steer 500 - 6 Power -> UTS Mini Mixing Desk - Compressor
