File: sidechain.kicad_sch (KiCad schematic)
At the start: 30 parts, among them SW2 INT/EXT, SW3 HPF DEFEAT, SW4 LINK, U3 NE5532, U4 NE5532, U6 NE5532

Commit message: add Docs & fix name & all the other shit
Other:
- company: Steer 500 -> UTS Mini Mixing Desk
- title: Steer 500 - 5 Sidechain -> UTS Mini Mixing Desk - Compressor
Changed lines of the file:
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@@
 	(paper "User" 393.7 194.31)
 	(title_block
-		(title "Steer 500 - 5 Sidechain")
+		(title "UTS Mini Mixing Desk - Compressor")
 		(date "2026-08-31")
 		(rev "A")
-		(company "Steer 500")
+		(company "UTS Mini Mixing Desk")
 	)
 	(junction
@@
 		)
 		(instances
-			(project "steer500-sections"
+			(project "UTS Mini Mixing Desk - Compressor"
 				(path "/fdeae63a-37f5-58fb-b342-cb68d8a6bfbc/726d8415-a5fc-52c7-823f-9ededf5a8991"
 					(reference "RV6")
@@
 		)
 		(instances
-			(project "steer500-sections"
+			(project "UTS Mini Mixing Desk - Compressor"
 				(path "/fdeae63a-37f5-58fb-b342-cb68d8a6bfbc/726d8415-a5fc-52c7-823f-9ededf5a8991"
 					(reference "R49")
@@
 		)
 		(instances
-			(project "steer500-sections"
+			(project "UTS Mini Mixing Desk - Compressor"
 				(path "/fdeae63a-37f5-58fb-b342-cb68d8a6bfbc/726d8415-a5fc-52c7-823f-9ededf5a8991"
 					(reference "SW4")
@@
 		)
 		(instances
-			(project "steer500-sections"
+			(project "UTS Mini Mixing Desk - Compressor"
 				(path "/fdeae63a-37f5-58fb-b342-cb68d8a6bfbc/726d8415-a5fc-52c7-823f-9ededf5a8991"
 					(reference "U3")
@@
 		)
 		(instances
-			(project "steer500-sections"
+			(project "UTS Mini Mixing Desk - Compressor"
 				(path "/fdeae63a-37f5-58fb-b342-cb68d8a6bfbc/726d8415-a5fc-52c7-823f-9ededf5a8991"
 					(reference "#PWRSI002")
@@
 		)
 		(instances
-			(project "steer500-sections"
+			(project "UTS Mini Mixing Desk - Compressor"
 				(path "/fdeae63a-37f5-58fb-b342-cb68d8a6bfbc/726d8415-a5fc-52c7-823f-9ededf5a8991"
 					(reference "U4")
@@
 		)
 		(instances
-			(project "steer500-sections"
+			(project "UTS Mini Mixing Desk - Compressor"
 				(path "/fdeae63a-37f5-58fb-b342-cb68d8a6bfbc/726d8415-a5fc-52c7-823f-9ededf5a8991"
 					(reference "#PWRSI003")
@@
 		)
 		(instances
-			(project "steer500-sections"
+			(project "UTS Mini Mixing Desk - Compressor"
 				(path "/fdeae63a-37f5-58fb-b342-cb68d8a6bfbc/726d8415-a5fc-52c7-823f-9ededf5a8991"
 					(reference "R35")
@@
 		)
 		(instances
-			(project "steer500-sections"
+			(project "UTS Mini Mixing Desk - Compressor"
 				(path "/fdeae63a-37f5-58fb-b342-cb68d8a6bfbc/726d8415-a5fc-52c7-823f-9ededf5a8991"
 					(reference "R44")
@@
 		)
 		(instances
-			(project "steer500-sections"
+			(project "UTS Mini Mixing Desk - Compressor"
 				(path "/fdeae63a-37f5-58fb-b342-cb68d8a6bfbc/726d8415-a5fc-52c7-823f-9ededf5a8991"
 					(reference "R42")
@@
 		)
 		(instances
-			(project "steer500-sections"
+			(project "UTS Mini Mixing Desk - Compressor"
 				(path "/fdeae63a-37f5-58fb-b342-cb68d8a6bfbc/726d8415-a5fc-52c7-823f-9ededf5a8991"
 					(reference "R74")
@@
 		)
 		(instances
-			(project "steer500-sections"
+			(project "UTS Mini Mixing Desk - Compressor"
 				(path "/fdeae63a-37f5-58fb-b342-cb68d8a6bfbc/726d8415-a5fc-52c7-823f-9ededf5a8991"
 					(reference "SW3")
@@
 		)
 		(instances
-			(project "steer500-sections"
+			(project "UTS Mini Mixing Desk - Compressor"
 				(path "/fdeae63a-37f5-58fb-b342-cb68d8a6bfbc/726d8415-a5fc-52c7-823f-9ededf5a8991"
 					(reference "R39")
@@
 		)
 		(instances
-			(project "steer500-sections"
+			(project "UTS Mini Mixing Desk - Compressor"
 				(path "/fdeae63a-37f5-58fb-b342-cb68d8a6bfbc/726d8415-a5fc-52c7-823f-9ededf5a8991"
 					(reference "SW2")
@@
 		)
 		(instances
-			(project "steer500-sections"
+			(project "UTS Mini Mixing Desk - Compressor"
 				(path "/fdeae63a-37f5-58fb-b342-cb68d8a6bfbc/726d8415-a5fc-52c7-823f-9ededf5a8991"
 					(reference "R45")
@@
 		)
 		(instances
-			(project "steer500-sections"
+			(project "UTS Mini Mixing Desk - Compressor"
 				(path "/fdeae63a-37f5-58fb-b342-cb68d8a6bfbc/726d8415-a5fc-52c7-823f-9ededf5a8991"
 					(reference "R47")
@@
 		)
 		(instances
-			(project "steer500-sections"
+			(project "UTS Mini Mixing Desk - Compressor"
 				(path "/fdeae63a-37f5-58fb-b342-cb68d8a6bfbc/726d8415-a5fc-52c7-823f-9ededf5a8991"
 					(reference "R46")
@@
 		)
 		(instances
-			(project "steer500-sections"
+			(project "UTS Mini Mixing Desk - Compressor"
 				(path "/fdeae63a-37f5-58fb-b342-cb68d8a6bfbc/726d8415-a5fc-52c7-823f-9ededf5a8991"
 					(reference "RV4")
@@
 		)
 		(instances
-			(project "steer500-sections"
+			(project "UTS Mini Mixing Desk - Compressor"
 				(path "/fdeae63a-37f5-58fb-b342-cb68d8a6bfbc/726d8415-a5fc-52c7-823f-9ededf5a8991"
 					(reference "R40")
@@
 		)
 		(instances
-			(project "steer500-sections"
+			(project "UTS Mini Mixing Desk - Compressor"
 				(path "/fdeae63a-37f5-58fb-b342-cb68d8a6bfbc/726d8415-a5fc-52c7-823f-9ededf5a8991"
 					(reference "U4")
@@
 		)
 		(instances
-			(project "steer500-sections"
+			(project "UTS Mini Mixing Desk - Compressor"
 				(path "/fdeae63a-37f5-58fb-b342-cb68d8a6bfbc/726d8415-a5fc-52c7-823f-9ededf5a8991"
 					(reference "U3")
@@
 		)
 		(instances
-			(project "steer500-sections"
+			(project "UTS Mini Mixing Desk - Compressor"
 				(path "/fdeae63a-37f5-58fb-b342-cb68d8a6bfbc/726d8415-a5fc-52c7-823f-9ededf5a8991"
 					(reference "R36")
@@
 		)
 		(instances
-			(project "steer500-sections"
+			(project "UTS Mini Mixing Desk - Compressor"
 				(path "/fdeae63a-37f5-58fb-b342-cb68d8a6bfbc/726d8415-a5fc-52c7-823f-9ededf5a8991"
 					(reference "D7")
@@
 		)
 		(instances
-			(project "steer500-sections"
+			(project "UTS Mini Mixing Desk - Compressor"
 				(path "/fdeae63a-37f5-58fb-b342-cb68d8a6bfbc/726d8415-a5fc-52c7-823f-9ededf5a8991"
 					(reference "#PWRSI006")
@@
 		)
 		(instances
-			(project "steer500-sections"
+			(project "UTS Mini Mixing Desk - Compressor"
 				(path "/fdeae63a-37f5-58fb-b342-cb68d8a6bfbc/726d8415-a5fc-52c7-823f-9ededf5a8991"
 					(reference "R38")
@@
 		)
 		(instances
-			(project "steer500-sections"
+			(project "UTS Mini Mixing Desk - Compressor"
 				(path "/fdeae63a-37f5-58fb-b342-cb68d8a6bfbc/726d8415-a5fc-52c7-823f-9ededf5a8991"
 					(reference "R37")
@@
 		)
 		(instances
-			(project "steer500-sections"
+			(project "UTS Mini Mixing Desk - Compressor"
 				(path "/fdeae63a-37f5-58fb-b342-cb68d8a6bfbc/726d8415-a5fc-52c7-823f-9ededf5a8991"
 					(reference "C15")
@@
 		)
 		(instances
-			(project "steer500-sections"
+			(project "UTS Mini Mixing Desk - Compressor"
 				(path "/fdeae63a-37f5-58fb-b342-cb68d8a6bfbc/726d8415-a5fc-52c7-823f-9ededf5a8991"
 					(reference "RV5")
@@
 		)
 		(instances
-			(project "steer500-sections"
+			(project "UTS Mini Mixing Desk - Compressor"
 				(path "/fdeae63a-37f5-58fb-b342-cb68d8a6bfbc/726d8415-a5fc-52c7-823f-9ededf5a8991"
 					(reference "RV3")
@@
 		)
 		(instances
-			(project "steer500-sections"
+			(project "UTS Mini Mixing Desk - Compressor"
 				(path "/fdeae63a-37f5-58fb-b342-cb68d8a6bfbc/726d8415-a5fc-52c7-823f-9ededf5a8991"
 					(reference "#PWRSI001")
@@
 		)
 		(instances
-			(project "steer500-sections"
+			(project "UTS Mini Mixing Desk - Compressor"
 				(path "/fdeae63a-37f5-58fb-b342-cb68d8a6bfbc/726d8415-a5fc-52c7-823f-9ededf5a8991"
 					(reference "#PWRSI000")
@@
 		)
 		(instances
-			(project "steer500-sections"
+			(project "UTS Mini Mixing Desk - Compressor"
 				(path "/fdeae63a-37f5-58fb-b342-cb68d8a6bfbc/726d8415-a5fc-52c7-823f-9ededf5a8991"
 					(reference "D5")
@@
 		)
 		(instances
-			(project "steer500-sections"
+			(project "UTS Mini Mixing Desk - Compressor"
 				(path "/fdeae63a-37f5-58fb-b342-cb68d8a6bfbc/726d8415-a5fc-52c7-823f-9ededf5a8991"
 					(reference "U6")
@@
 		)
 		(instances
-			(project "steer500-sections"
+			(project "UTS Mini Mixing Desk - Compressor"
 				(path "/fdeae63a-37f5-58fb-b342-cb68d8a6bfbc/726d8415-a5fc-52c7-823f-9ededf5a8991"
 					(reference "#PWRSI005")
@@
 		)
 		(instances
-			(project "steer500-sections"
+			(project "UTS Mini Mixing Desk - Compressor"
 				(path "/fdeae63a-37f5-58fb-b342-cb68d8a6bfbc/726d8415-a5fc-52c7-823f-9ededf5a8991"
 					(reference "R41")
@@
 		)
 		(instances
-			(project "steer500-sections"
+			(project "UTS Mini Mixing Desk - Compressor"
 				(path "/fdeae63a-37f5-58fb-b342-cb68d8a6bfbc/726d8415-a5fc-52c7-823f-9ededf5a8991"
 					(reference "#PWRSI004")
@@
 		)
 		(instances
-			(project "steer500-sections"
+			(project "UTS Mini Mixing Desk - Compressor"
 				(path "/fdeae63a-37f5-58fb-b342-cb68d8a6bfbc/726d8415-a5fc-52c7-823f-9ededf5a8991"
 					(reference "R43")
@@
 		)
 		(instances
-			(project "steer500-sections"
+			(project "UTS Mini Mixing Desk - Compressor"
 				(path "/fdeae63a-37f5-58fb-b342-cb68d8a6bfbc/726d8415-a5fc-52c7-823f-9ededf5a8991"
 					(reference "C14")
@@
 		)
 		(instances
-			(project "steer500-sections"
+			(project "UTS Mini Mixing Desk - Compressor"
 				(path "/fdeae63a-37f5-58fb-b342-cb68d8a6bfbc/726d8415-a5fc-52c7-823f-9ededf5a8991"
 					(reference "D6")
