File: vca.kicad_sch (KiCad schematic)
At the start: 29 parts, among them Q1 BC549C, Q2 BC549C, Q3 BC549C, Q4 BC549C, Q5 BC549C, Q6 BC549C, Q7 BC549C, Q8 BC549C, Q9 BC549C, U1 NE5532

Commit message: add Docs & fix name & all the other shit
Connections:
- net at Q3.1 (C), R14.2, R15.2: now also Q2.1 (C), Q8.3 (E), Q9.3 (E)
- net at C9.1, Q4.3 (E), R19.1: now also C9.2, R21.1
Other:
- company: Steer 500 -> UTS Mini Mixing Desk
- title: Steer 500 - 3 VCA -> UTS Mini Mixing Desk - Compressor
- moved on the sheet: C10, C11, C5, C8, C9, Q1, Q2, Q3, Q4, Q5, Q6, Q7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

Commit message: Add cool graphics
Connections:
- net at Q3.1 (C), R14.2, R15.2: no longer Q2.1 (C), Q8.3 (E), Q9.3 (E)
- net at C9.1, Q4.3 (E), R19.1: no longer C9.2, R21.1
- new net: Q2.1 (C), Q8.3 (E), Q9.3 (E)
- new net: C9.2, R21.1
Other:
- moved on the sheet: R14
Changed lines of the file:
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@@
 	)
 	(junction
-		(at 99.06 72.39)
-		(diameter 0)
-		(color 0 0 0 0)
-	)
-	(junction
 		(at 121.92 82.55)
 		(diameter 0)
@@
 	)
 	(junction
-		(at 177.8 133.35)
+		(at 215.9 123.19)
 		(diameter 0)
 		(color 0 0 0 0)
 	)
 	(junction
-		(at 215.9 123.19)
+		(at 99.06 72.39)
 		(diameter 0)
 		(color 0 0 0 0)
@@
 	)
 	(junction
-		(at 85.09 72.39)
-		(diameter 0)
-		(color 0 0 0 0)
-	)
-	(junction
 		(at 175.26 31.75)
 		(diameter 0)
@@
 	)
 	(junction
-		(at 177.8 125.73)
-		(diameter 0)
-		(color 0 0 0 0)
-	)
-	(junction
 		(at 177.8 123.19)
 		(diameter 0)
@@
 	(wire
 		(pts
-			(xy 55.88 72.39) (xy 77.47 72.39)
+			(xy 55.88 72.39) (xy 68.58 72.39)
 		)
 		(stroke
@@
 	(wire
 		(pts
-			(xy 177.8 133.35) (xy 177.8 125.73)
+			(xy 101.6 50.8) (xy 101.6 59.69)
 		)
 		(stroke
@@
 	(wire
 		(pts
-			(xy 101.6 50.8) (xy 101.6 59.69)
+			(xy 85.09 38.1) (xy 101.6 38.1)
 		)
 		(stroke
@@
 	(wire
 		(pts
-			(xy 85.09 38.1) (xy 101.6 38.1)
+			(xy 205.74 109.22) (xy 208.28 109.22)
 		)
 		(stroke
@@
 	(wire
 		(pts
-			(xy 205.74 109.22) (xy 208.28 109.22)
+			(xy 85.09 38.1) (xy 85.09 116.84)
 		)
 		(stroke
@@
 	(wire
 		(pts
-			(xy 85.09 38.1) (xy 85.09 72.39)
+			(xy 72.39 45.72) (xy 93.98 45.72)
 		)
 		(stroke
@@
 	(wire
 		(pts
-			(xy 72.39 45.72) (xy 93.98 45.72)
+			(xy 34.29 60.96) (xy 31.75 60.96)
 		)
 		(stroke
@@
 	(wire
 		(pts
-			(xy 34.29 60.96) (xy 31.75 60.96)
+			(xy 121.92 111.76) (xy 127 111.76)
 		)
 		(stroke
@@
 	(wire
 		(pts
-			(xy 121.92 111.76) (xy 127 111.76)
+			(xy 76.2 72.39) (xy 99.06 72.39)
 		)
 		(stroke
@@
 	(wire
 		(pts
-			(xy 85.09 72.39) (xy 99.06 72.39)
-		)
-		(stroke
-			(width 0)
-			(type default)
-		)
-	)
-	(wire
-		(pts
 			(xy 40.64 68.58) (xy 44.45 68.58)
 		)
@@
 	(wire
 		(pts
-			(xy 85.09 72.39) (xy 85.09 116.84)
-		)
-		(stroke
-			(width 0)
-			(type default)
-		)
-	)
-	(wire
-		(pts
 			(xy 177.8 50.8) (xy 177.8 54.61)
 		)
@@
 	(symbol
 		(lib_id "Device:R")
-		(at 81.28 72.39 90)
+		(at 72.39 72.39 90)
 		(unit 1)
 		(exclude_from_sim no)
@@
 		(dnp no)
 		(property "Reference" "R14"
-			(at 80.01 68.58 0)
+			(at 71.12 68.58 0)
 			(effects
 				(font
@@
 		)
 		(property "Value" "220R"
-			(at 83.18 68.58 0)
+			(at 74.29 68.58 0)
 			(effects
 				(font
@@
 		)
 		(property "Footprint" "Resistor_THT:R_Axial_DIN0207_L6.3mm_D2.5mm_P10.16mm_Horizontal"
-			(at 81.28 72.39 0)
+			(at 72.39 72.39 0)
 			(effects
 				(font
@@
 		)
 		(property "Datasheet" ""
-			(at 81.28 72.39 0)
+			(at 72.39 72.39 0)
 			(effects
 				(font
@@
 		)
 		(property "Description" ""
-			(at 81.28 72.39 0)
+			(at 72.39 72.39 0)
 			(effects
 				(font
