File: kicad_withpcb/compressor_with_pcb/compressor_with_pcb.kicad_pcb (KiCad board)
At the start: 2 copper layers, 152.3 x 105 mm, 1 part, among them J1 EDA 306

Commit message: Fix issues with schematic and basic add pcb
Parts:
- added C1: 22u, Capacitor_THT:CP_Radial_D6.3mm_P2.50mm, F.Cu at (154.5, 83.3)
- added C10: 2u2, Capacitor_THT:C_Rect_L7.0mm_W2.5mm_P5.00mm, F.Cu at (154.4, 129.9)
- added C11: 100p, Capacitor_THT:C_Disc_D5.0mm_W2.5mm_P5.00mm, F.Cu at (129.8, 129.9)
- added C13: 100p, Capacitor_THT:C_Disc_D5.0mm_W2.5mm_P5.00mm, F.Cu at (129.8, 134.0)
- added C14: 220n, Capacitor_THT:C_Rect_L7.0mm_W2.5mm_P5.00mm, F.Cu at (154.4, 134.0)
- added C15: 10u, Capacitor_THT:C_Rect_L7.0mm_W2.5mm_P5.00mm, F.Cu at (154.4, 138.0)
- added C16: 100u, Capacitor_THT:CP_Radial_D6.3mm_P2.50mm, F.Cu at (162.4, 83.3)
- added C17: 100u, Capacitor_THT:CP_Radial_D6.3mm_P2.50mm, F.Cu at (162.4, 91.2)
- added C18: 10n, Capacitor_THT:C_Disc_D5.0mm_W2.5mm_P5.00mm, F.Cu at (129.8, 138.0)
- added C19: 47u, Capacitor_THT:CP_Radial_D6.3mm_P2.50mm, F.Cu at (162.4, 99.0)
- added C2: 22u, Capacitor_THT:CP_Radial_D6.3mm_P2.50mm, F.Cu at (154.5, 91.2)
- added C20: 100n, Capacitor_THT:C_Disc_D5.0mm_W2.5mm_P5.00mm, F.Cu at (129.8, 142.1)
- added C21: 47u, Capacitor_THT:CP_Radial_D6.3mm_P2.50mm, F.Cu at (170.4, 83.3)
- added C22: 47u, Capacitor_THT:CP_Radial_D6.3mm_P2.50mm, F.Cu at (170.4, 91.2)
- added C23: 100n, Capacitor_THT:C_Disc_D5.0mm_W2.5mm_P5.00mm, F.Cu at (129.8, 146.1)
- added C24: 100n, Capacitor_THT:C_Disc_D5.0mm_W2.5mm_P5.00mm, F.Cu at (137.9, 117.8)
- added C25: 100n, Capacitor_THT:C_Disc_D5.0mm_W2.5mm_P5.00mm, F.Cu at (137.9, 121.8)
- added C26: 100n, Capacitor_THT:C_Disc_D5.0mm_W2.5mm_P5.00mm, F.Cu at (137.9, 125.9)
- added C27: 100n, Capacitor_THT:C_Disc_D5.0mm_W2.5mm_P5.00mm, F.Cu at (137.9, 129.9)
- added C28: 100n, Capacitor_THT:C_Disc_D5.0mm_W2.5mm_P5.00mm, F.Cu at (137.9, 134.0)
- added C29: 100n, Capacitor_THT:C_Disc_D5.0mm_W2.5mm_P5.00mm, F.Cu at (137.9, 138.0)
- added C3: 1n, Capacitor_THT:C_Disc_D5.0mm_W2.5mm_P5.00mm, F.Cu at (129.8, 117.8)
- added C30: 100n, Capacitor_THT:C_Disc_D5.0mm_W2.5mm_P5.00mm, F.Cu at (137.9, 142.1)
- added C31: 100n, Capacitor_THT:C_Disc_D5.0mm_W2.5mm_P5.00mm, F.Cu at (137.9, 146.1)
- added C32: 100n, Capacitor_THT:C_Disc_D5.0mm_W2.5mm_P5.00mm, F.Cu at (146.1, 117.8)
- added C33: 100n, Capacitor_THT:C_Disc_D5.0mm_W2.5mm_P5.00mm, F.Cu at (146.1, 121.8)
- added C34: 100n, Capacitor_THT:C_Disc_D5.0mm_W2.5mm_P5.00mm, F.Cu at (146.1, 125.9)
- added C35: 2u2, Capacitor_THT:C_Rect_L7.0mm_W2.5mm_P5.00mm, F.Cu at (154.4, 142.1)
- added C36: 100n, Capacitor_THT:C_Disc_D5.0mm_W2.5mm_P5.00mm, F.Cu at (146.1, 129.9)
- added C37: 100n, Capacitor_THT:C_Disc_D5.0mm_W2.5mm_P5.00mm, F.Cu at (146.1, 134.0)
- added C38: 47u, Capacitor_THT:CP_Radial_D6.3mm_P2.50mm, F.Cu at (170.4, 99.0)
- added C4: 1n, Capacitor_THT:C_Disc_D5.0mm_W2.5mm_P5.00mm, F.Cu at (129.8, 121.8)
- added C41: 100n, Capacitor_THT:C_Disc_D5.0mm_W2.5mm_P5.00mm, F.Cu at (146.1, 138.0)
- added C42: 100n, Capacitor_THT:C_Disc_D5.0mm_W2.5mm_P5.00mm, F.Cu at (146.1, 142.1)
- added C5: 10u, Capacitor_THT:C_Rect_L7.0mm_W2.5mm_P5.00mm, F.Cu at (154.4, 117.8)
- added C6: 100u, Capacitor_THT:CP_Radial_D6.3mm_P2.50mm, F.Cu at (154.5, 99.0)
- added C7: 100n, Capacitor_THT:C_Disc_D5.0mm_W2.5mm_P5.00mm, F.Cu at (129.8, 125.9)
- added C8: 10u, Capacitor_THT:C_Rect_L7.0mm_W2.5mm_P5.00mm, F.Cu at (154.4, 121.8)
- added C9: 2u2, Capacitor_THT:C_Rect_L7.0mm_W2.5mm_P5.00mm, F.Cu at (154.4, 125.9)
- added D10: BZX79-C5V1, Diode_THT:D_DO-35_SOD27_P7.62mm_Horizontal, F.Cu at (104.3, 151.6)
- added D11: 1N4148, Diode_THT:D_DO-35_SOD27_P7.62mm_Horizontal, F.Cu at (104.3, 155.1)
- added D12: 1N4148, Diode_THT:D_DO-35_SOD27_P7.62mm_Horizontal, F.Cu at (104.3, 158.7)
- added D20: meter, LED_THT:LED_D2.0mm_W4.0mm_H2.8mm_FlatTop, F.Cu at (86.8, 141.4)
- added D21: meter, LED_THT:LED_D2.0mm_W4.0mm_H2.8mm_FlatTop, F.Cu at (86.8, 145.9)
- added D22: meter, LED_THT:LED_D2.0mm_W4.0mm_H2.8mm_FlatTop, F.Cu at (86.8, 150.3)
- added D23: meter, LED_THT:LED_D2.0mm_W4.0mm_H2.8mm_FlatTop, F.Cu at (86.8, 154.8)
- added D24: meter, LED_THT:LED_D2.0mm_W4.0mm_H2.8mm_FlatTop, F.Cu at (86.8, 159.3)
- added D25: meter, LED_THT:LED_D2.0mm_W4.0mm_H2.8mm_FlatTop, F.Cu at (92.7, 141.4)
- added D26: meter, LED_THT:LED_D2.0mm_W4.0mm_H2.8mm_FlatTop, F.Cu at (92.7, 145.9)
- added D30: meter, LED_THT:LED_D2.0mm_W4.0mm_H2.8mm_FlatTop, F.Cu at (92.7, 150.3)
- added D31: meter, LED_THT:LED_D2.0mm_W4.0mm_H2.8mm_FlatTop, F.Cu at (92.7, 154.8)
- added D32: meter, LED_THT:LED_D2.0mm_W4.0mm_H2.8mm_FlatTop, F.Cu at (92.7, 159.3)
- added D33: meter, LED_THT:LED_D2.0mm_W4.0mm_H2.8mm_FlatTop, F.Cu at (98.6, 141.4)
- added D34: meter, LED_THT:LED_D2.0mm_W4.0mm_H2.8mm_FlatTop, F.Cu at (98.6, 145.9)
- added D35: meter, LED_THT:LED_D2.0mm_W4.0mm_H2.8mm_FlatTop, F.Cu at (98.6, 150.3)
- added D36: meter, LED_THT:LED_D2.0mm_W4.0mm_H2.8mm_FlatTop, F.Cu at (98.6, 154.8)
- added D5: 1N4148, Diode_THT:D_DO-35_SOD27_P7.62mm_Horizontal, F.Cu at (104.3, 140.9)
- added D6: 1N4148, Diode_THT:D_DO-35_SOD27_P7.62mm_Horizontal, F.Cu at (104.3, 144.5)
- added D7: 1N4148, Diode_THT:D_DO-35_SOD27_P7.62mm_Horizontal, F.Cu at (104.3, 148.0)
- added D8: 1N4004, Diode_THT:D_DO-41_SOD81_P7.62mm_Horizontal, F.Cu at (130.1, 150.3)
- added D9: 1N4004, Diode_THT:D_DO-41_SOD81_P7.62mm_Horizontal, F.Cu at (130.1, 154.5)
- added LED1: GR, LED_THT:LED_D3.0mm, F.Cu at (141.3, 150.9)
- added Q1: BC549C, Package_TO_SOT_THT:TO-92_Inline, F.Cu at (154.7, 147.4)
- added Q2: BC549C, Package_TO_SOT_THT:TO-92_Inline, F.Cu at (154.7, 153.1)
- added Q3: BC549C, Package_TO_SOT_THT:TO-92_Inline, F.Cu at (154.7, 158.9)
- added Q4: BC549C, Package_TO_SOT_THT:TO-92_Inline, F.Cu at (161.2, 147.4)
- added Q5: BC549C, Package_TO_SOT_THT:TO-92_Inline, F.Cu at (161.2, 153.1)
- added Q6: BC549C, Package_TO_SOT_THT:TO-92_Inline, F.Cu at (161.2, 158.9)
- added Q7: BC549C, Package_TO_SOT_THT:TO-92_Inline, F.Cu at (167.7, 147.4)
- added Q8: BC549C, Package_TO_SOT_THT:TO-92_Inline, F.Cu at (167.7, 153.1)
- added Q9: BC549C, Package_TO_SOT_THT:TO-92_Inline, F.Cu at (167.7, 158.9)
- added R1: 22k, Resistor_THT:R_Axial_DIN0207_L6.3mm_D2.5mm_P10.16mm_Horizontal, F.Cu at (86.7, 57.0)
- added R10: 11k, Resistor_THT:R_Axial_DIN0207_L6.3mm_D2.5mm_P10.16mm_Horizontal, F.Cu at (86.7, 93.5)
- added R11: 10k, Resistor_THT:R_Axial_DIN0207_L6.3mm_D2.5mm_P10.16mm_Horizontal, F.Cu at (86.7, 97.5)
- added R12: 10k, Resistor_THT:R_Axial_DIN0207_L6.3mm_D2.5mm_P10.16mm_Horizontal, F.Cu at (86.7, 101.6)
- added R13: 220R, Resistor_THT:R_Axial_DIN0207_L6.3mm_D2.5mm_P10.16mm_Horizontal, F.Cu at (86.7, 105.6)
- added R14: 220R, Resistor_THT:R_Axial_DIN0207_L6.3mm_D2.5mm_P10.16mm_Horizontal, F.Cu at (86.7, 109.7)
- added R15: 220R, Resistor_THT:R_Axial_DIN0207_L6.3mm_D2.5mm_P10.16mm_Horizontal, F.Cu at (86.7, 113.7)
- added R16: 4k7, Resistor_THT:R_Axial_DIN0207_L6.3mm_D2.5mm_P10.16mm_Horizontal, F.Cu at (100.0, 57.0)
- added R17: 4k7, Resistor_THT:R_Axial_DIN0207_L6.3mm_D2.5mm_P10.16mm_Horizontal, F.Cu at (100.0, 61.1)
- added R18: 1k5, Resistor_THT:R_Axial_DIN0207_L6.3mm_D2.5mm_P10.16mm_Horizontal, F.Cu at (100.0, 65.1)
- added R19: 10k, Resistor_THT:R_Axial_DIN0207_L6.3mm_D2.5mm_P10.16mm_Horizontal, F.Cu at (100.0, 69.2)
- added R2: 22k, Resistor_THT:R_Axial_DIN0207_L6.3mm_D2.5mm_P10.16mm_Horizontal, F.Cu at (86.7, 61.1)
- added R20: 10k, Resistor_THT:R_Axial_DIN0207_L6.3mm_D2.5mm_P10.16mm_Horizontal, F.Cu at (100.0, 73.2)
- added R21: 3k3, Resistor_THT:R_Axial_DIN0207_L6.3mm_D2.5mm_P10.16mm_Horizontal, F.Cu at (100.0, 77.3)
- added R22: 3k3, Resistor_THT:R_Axial_DIN0207_L6.3mm_D2.5mm_P10.16mm_Horizontal, F.Cu at (100.0, 81.3)
- added R23: 22k, Resistor_THT:R_Axial_DIN0207_L6.3mm_D2.5mm_P10.16mm_Horizontal, F.Cu at (100.0, 85.4)
- added R24: 22k, Resistor_THT:R_Axial_DIN0207_L6.3mm_D2.5mm_P10.16mm_Horizontal, F.Cu at (100.0, 89.4)
- added R26: 1k, Resistor_THT:R_Axial_DIN0207_L6.3mm_D2.5mm_P10.16mm_Horizontal, F.Cu at (100.0, 93.5)
- added R28: 100R, Resistor_THT:R_Axial_DIN0207_L6.3mm_D2.5mm_P10.16mm_Horizontal, F.Cu at (100.0, 97.5)
- added R29: 10k, Resistor_THT:R_Axial_DIN0207_L6.3mm_D2.5mm_P10.16mm_Horizontal, F.Cu at (100.0, 101.6)
- added R3: 22k, Resistor_THT:R_Axial_DIN0207_L6.3mm_D2.5mm_P10.16mm_Horizontal, F.Cu at (86.7, 65.1)
- added R30: 10k, Resistor_THT:R_Axial_DIN0207_L6.3mm_D2.5mm_P10.16mm_Horizontal, F.Cu at (100.0, 105.6)
- added R31: 5k1, Resistor_THT:R_Axial_DIN0207_L6.3mm_D2.5mm_P10.16mm_Horizontal, F.Cu at (100.0, 109.7)
- added R32: 100R, Resistor_THT:R_Axial_DIN0207_L6.3mm_D2.5mm_P10.16mm_Horizontal, F.Cu at (100.0, 113.7)
- added R33: 100R, Resistor_THT:R_Axial_DIN0207_L6.3mm_D2.5mm_P10.16mm_Horizontal, F.Cu at (113.3, 57.0)
- added R34: 100R, Resistor_THT:R_Axial_DIN0207_L6.3mm_D2.5mm_P10.16mm_Horizontal, F.Cu at (113.3, 61.1)
- added R35: 20k, Resistor_THT:R_Axial_DIN0207_L6.3mm_D2.5mm_P10.16mm_Horizontal, F.Cu at (113.3, 65.1)
- added R36: 100k, Resistor_THT:R_Axial_DIN0207_L6.3mm_D2.5mm_P10.16mm_Horizontal, F.Cu at (113.3, 69.2)
- added R37: 47k, Resistor_THT:R_Axial_DIN0207_L6.3mm_D2.5mm_P10.16mm_Horizontal, F.Cu at (113.3, 73.2)
- added R38: 10k, Resistor_THT:R_Axial_DIN0207_L6.3mm_D2.5mm_P10.16mm_Horizontal, F.Cu at (113.3, 77.3)
- added R39: 10k, Resistor_THT:R_Axial_DIN0207_L6.3mm_D2.5mm_P10.16mm_Horizontal, F.Cu at (113.3, 81.3)
- added R4: 22k, Resistor_THT:R_Axial_DIN0207_L6.3mm_D2.5mm_P10.16mm_Horizontal, F.Cu at (86.7, 69.2)
- added R40: 10k, Resistor_THT:R_Axial_DIN0207_L6.3mm_D2.5mm_P10.16mm_Horizontal, F.Cu at (113.3, 85.4)
- added R41: 10k, Resistor_THT:R_Axial_DIN0207_L6.3mm_D2.5mm_P10.16mm_Horizontal, F.Cu at (113.3, 89.4)
- added R42: 20k, Resistor_THT:R_Axial_DIN0207_L6.3mm_D2.5mm_P10.16mm_Horizontal, F.Cu at (113.3, 93.5)
- added R43: 10k, Resistor_THT:R_Axial_DIN0207_L6.3mm_D2.5mm_P10.16mm_Horizontal, F.Cu at (113.3, 97.5)
- added R44: 20k, Resistor_THT:R_Axial_DIN0207_L6.3mm_D2.5mm_P10.16mm_Horizontal, F.Cu at (113.3, 101.6)
- added R45: 220R, Resistor_THT:R_Axial_DIN0207_L6.3mm_D2.5mm_P10.16mm_Horizontal, F.Cu at (113.3, 105.6)
- added R46: 47R, Resistor_THT:R_Axial_DIN0207_L6.3mm_D2.5mm_P10.16mm_Horizontal, F.Cu at (113.3, 109.7)
- added R47: 4k7, Resistor_THT:R_Axial_DIN0207_L6.3mm_D2.5mm_P10.16mm_Horizontal, F.Cu at (113.3, 113.7)
- added R48: 0R, Resistor_THT:R_Axial_DIN0207_L6.3mm_D2.5mm_P10.16mm_Horizontal, F.Cu at (126.6, 57.0)
- added R49: 5k1, Resistor_THT:R_Axial_DIN0207_L6.3mm_D2.5mm_P10.16mm_Horizontal, F.Cu at (126.6, 61.1)
- added R5: 100R, Resistor_THT:R_Axial_DIN0207_L6.3mm_D2.5mm_P10.16mm_Horizontal, F.Cu at (86.7, 73.2)
- added R50: 10R, Resistor_THT:R_Axial_DIN0207_L6.3mm_D2.5mm_P10.16mm_Horizontal, F.Cu at (126.6, 65.1)
- added R51: 10R, Resistor_THT:R_Axial_DIN0207_L6.3mm_D2.5mm_P10.16mm_Horizontal, F.Cu at (126.6, 69.2)
- added R52: 100R, Resistor_THT:R_Axial_DIN0207_L6.3mm_D2.5mm_P10.16mm_Horizontal, F.Cu at (126.6, 73.2)
- added R53: 1k8, Resistor_THT:R_Axial_DIN0207_L6.3mm_D2.5mm_P10.16mm_Horizontal, F.Cu at (126.6, 77.3)
- added R6: 100R, Resistor_THT:R_Axial_DIN0207_L6.3mm_D2.5mm_P10.16mm_Horizontal, F.Cu at (86.7, 77.3)
- added R60: 47k, Resistor_THT:R_Axial_DIN0207_L6.3mm_D2.5mm_P10.16mm_Horizontal, F.Cu at (126.6, 81.3)
- added R61: 1k33, Resistor_THT:R_Axial_DIN0207_L6.3mm_D2.5mm_P10.16mm_Horizontal, F.Cu at (126.6, 85.4)
- added R62: 23k2, Resistor_THT:R_Axial_DIN0207_L6.3mm_D2.5mm_P10.16mm_Horizontal, F.Cu at (126.6, 89.4)
- added R68: 1k, Resistor_THT:R_Axial_DIN0207_L6.3mm_D2.5mm_P10.16mm_Horizontal, F.Cu at (126.6, 93.5)
- added R69: 36k, Resistor_THT:R_Axial_DIN0207_L6.3mm_D2.5mm_P10.16mm_Horizontal, F.Cu at (126.6, 97.5)
- added R7: 8k2, Resistor_THT:R_Axial_DIN0207_L6.3mm_D2.5mm_P10.16mm_Horizontal, F.Cu at (86.7, 81.3)
- added R74: 220k, Resistor_THT:R_Axial_DIN0207_L6.3mm_D2.5mm_P10.16mm_Horizontal, F.Cu at (126.6, 101.6)
- added R77: 3k9, Resistor_THT:R_Axial_DIN0207_L6.3mm_D2.5mm_P10.16mm_Horizontal, F.Cu at (126.6, 105.6)
- added R8: 75R, Resistor_THT:R_Axial_DIN0207_L6.3mm_D2.5mm_P10.16mm_Horizontal, F.Cu at (86.7, 85.4)
- added R80: 22k, Resistor_THT:R_Axial_DIN0207_L6.3mm_D2.5mm_P10.16mm_Horizontal, F.Cu at (126.6, 109.7)
- added R81: 22k, Resistor_THT:R_Axial_DIN0207_L6.3mm_D2.5mm_P10.16mm_Horizontal, F.Cu at (126.6, 113.7)
- added R82: 22k, Resistor_THT:R_Axial_DIN0207_L6.3mm_D2.5mm_P10.16mm_Horizontal, F.Cu at (139.9, 57.0)
- added R83: 22k, Resistor_THT:R_Axial_DIN0207_L6.3mm_D2.5mm_P10.16mm_Horizontal, F.Cu at (139.9, 61.1)
- added R84: 10k, Resistor_THT:R_Axial_DIN0207_L6.3mm_D2.5mm_P10.16mm_Horizontal, F.Cu at (139.9, 65.1)
- added R85: 10k, Resistor_THT:R_Axial_DIN0207_L6.3mm_D2.5mm_P10.16mm_Horizontal, F.Cu at (139.9, 69.2)
- added R86: 10k, Resistor_THT:R_Axial_DIN0207_L6.3mm_D2.5mm_P10.16mm_Horizontal, F.Cu at (139.9, 73.2)
- added R87: 1k, Resistor_THT:R_Axial_DIN0207_L6.3mm_D2.5mm_P10.16mm_Horizontal, F.Cu at (139.9, 77.3)
- added R88: 100k, Resistor_THT:R_Axial_DIN0207_L6.3mm_D2.5mm_P10.16mm_Horizontal, F.Cu at (139.9, 81.3)
- added R89: 2k7, Resistor_THT:R_Axial_DIN0207_L6.3mm_D2.5mm_P10.16mm_Horizontal, F.Cu at (139.9, 85.4)
- added R9: 68k, Resistor_THT:R_Axial_DIN0207_L6.3mm_D2.5mm_P10.16mm_Horizontal, F.Cu at (86.7, 89.4)
- added R90: 8k2, Resistor_THT:R_Axial_DIN0207_L6.3mm_D2.5mm_P10.16mm_Horizontal, F.Cu at (139.9, 89.4)
- added R91: 2k7, Resistor_THT:R_Axial_DIN0207_L6.3mm_D2.5mm_P10.16mm_Horizontal, F.Cu at (139.9, 93.5)
- added R92: 8k2, Resistor_THT:R_Axial_DIN0207_L6.3mm_D2.5mm_P10.16mm_Horizontal, F.Cu at (139.9, 97.5)
- added R93: 18k, Resistor_THT:R_Axial_DIN0207_L6.3mm_D2.5mm_P10.16mm_Horizontal, F.Cu at (139.9, 101.6)
- added R94: 10k, Resistor_THT:R_Axial_DIN0207_L6.3mm_D2.5mm_P10.16mm_Horizontal, F.Cu at (139.9, 105.6)
- added RV1: 2k, Potentiometer_THT:Potentiometer_Bourns_3296W_Vertical, F.Cu at (121.6, 142.4)
- added RV2: 10k, Potentiometer_THT:Potentiometer_Alps_RK09K_Single_Vertical, F.Cu at (71.3, 59.7)
- added RV3: 1M, Potentiometer_THT:Potentiometer_Alps_RK09K_Single_Vertical, F.Cu at (71.3, 74.0)
- added RV4: 100k, Potentiometer_THT:Potentiometer_Alps_RK09K_Single_Vertical, F.Cu at (71.3, 88.4)
- added RV5: 4k7, Potentiometer_THT:Potentiometer_Alps_RK09K_Single_Vertical, F.Cu at (71.3, 102.7)
- added RV6: 220k, Potentiometer_THT:Potentiometer_Alps_RK09K_Single_Vertical, F.Cu at (71.3, 117.1)
- added RV7: 20k, Potentiometer_THT:Potentiometer_Bourns_3296W_Vertical, F.Cu at (121.6, 148.7)
- added RV8: 20k, Potentiometer_THT:Potentiometer_Bourns_3296W_Vertical, F.Cu at (121.6, 155.1)
- added U1: NE5532, Package_DIP:DIP-8_W7.62mm, F.Cu at (86.7, 117.8)
- added U10: LM3915, Package_DIP:DIP-18_W7.62mm, F.Cu at (164.0, 57.0)
- added U2: NE5532, Package_DIP:DIP-8_W7.62mm, F.Cu at (97.5, 117.8)
- added U3: NE5532, Package_DIP:DIP-8_W7.62mm, F.Cu at (108.2, 117.8)
- added U4: TL072, Package_DIP:DIP-8_W7.62mm, F.Cu at (119.0, 117.8)
- added U5: NE5532, Package_DIP:DIP-8_W7.62mm, F.Cu at (86.7, 129.5)
- added U6: NE5532, Package_DIP:DIP-8_W7.62mm, F.Cu at (97.5, 129.5)
- added U7: NE5532, Package_DIP:DIP-8_W7.62mm, F.Cu at (108.2, 129.5)
- added U9: LM3914, Package_DIP:DIP-18_W7.62mm, F.Cu at (153.2, 57.0)
Connections:
- net +48V renamed +48V-IN
- net /+OUT+4 renamed OUT+
- net /-OUT renamed OUT-
- net /SC_LINK renamed LINK
- J1 pad 1: /CHASSIS -> CHASSIS
- J1 pad 10: /+IN+4 -> IN+
- J1 pad 11: /GAIN_ADJ -> AUXIN+
- J1 pad 12: +16V -> +16V-IN
- J1 pad 13: GND -> PGND
- J1 pad 14: -16V -> -16V-IN
- J1 pad 3: /+OUT-2 -> AUXOUT+
- J1 pad 5: /AGND -> AGND
- J1 pad 7: /-IN-2 -> AUXOUT-
- J1 pad 8: /-IN+4 -> IN-
- J1 pad 9: /+IN-2 -> AUXIN-

Commit message: Add last few footprints for switches as header pins
Parts:
- added SW1: BYPASS, Connector_PinSocket_1.00mm:PinSocket_1x06_P1.00mm_Vertical, F.Cu at (169.2, 123.8)
- added SW2: INT/EXT, Connector_PinSocket_1.00mm:PinSocket_1x03_P1.00mm_Vertical, F.Cu at (180.2, 123.8)
- added SW3: HPF DEFEAT, Connector_PinSocket_1.00mm:PinSocket_1x02_P1.00mm_Vertical, F.Cu at (172.8, 123.8)
- added SW4: LINK, Connector_PinSocket_1.00mm:PinSocket_1x02_P1.00mm_Vertical, F.Cu at (176.3, 123.8)

Commit message: Finish Schematic re-organisation and begin pcb
Connections:
- C10 pad 1: Net-(Q5-E) -> Net-(C10-Pad1)
- C10 pad 2: Net-(C10-Pad2) -> Net-(Q5-E)
- C13 pad 1: Net-(U2B--) -> Net-(C13-Pad1)
- C13 pad 2: Net-(C13-Pad2) -> Net-(U2B--)
- Q3 pad 1: Net-(Q3-C) -> Net-(Q2-C)
- R14 pad 1: Net-(Q1-E) -> Net-(Q2-C)
- R14 pad 2: Net-(Q3-C) -> Net-(Q1-E)
- R15 pad 2: Net-(Q3-C) -> Net-(Q2-C)
- R22 pad 1: Net-(C10-Pad2) -> Net-(C10-Pad1)
- R30 pad 1: Net-(U2B--) -> Net-(C13-Pad1)
- R30 pad 2: Net-(C13-Pad2) -> Net-(U2B--)
- R32 pad 1: Net-(C13-Pad2) -> Net-(C13-Pad1)
- R7 pad 1: Net-(R4-Pad2) -> Net-(R7-Pad1)
- R7 pad 2: Net-(R7-Pad2) -> Net-(R4-Pad2)
- R82 pad 1: Net-(U5A--) -> KEY
- R82 pad 2: KEY -> Net-(U5A--)
- RV1 pad 1: Net-(R7-Pad2) -> Net-(R7-Pad1)
- U2 pad 7: Net-(C13-Pad2) -> Net-(C13-Pad1)
Changed lines of the file:
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@@
 			(layers "*.Cu" "*.Mask")
 			(remove_unused_layers no)
-			(net "Net-(C10-Pad2)")
+			(net "Net-(C10-Pad1)")
 			(pintype "passive")
 		)
@@
 			(layers "*.Cu" "*.Mask")
 			(remove_unused_layers no)
-			(net "Net-(C13-Pad2)")
+			(net "Net-(C13-Pad1)")
 			(pintype "passive")
 		)
@@
 			(layers "*.Cu" "*.Mask")
 			(remove_unused_layers no)
-			(net "Net-(Q1-E)")
+			(net "Net-(Q2-C)")
 			(pintype "passive")
 		)
@@
 			(layers "*.Cu" "*.Mask")
 			(remove_unused_layers no)
-			(net "Net-(Q3-C)")
+			(net "Net-(Q1-E)")
 			(pintype "passive")
 		)
@@
 			(layers "*.Cu" "*.Mask")
 			(remove_unused_layers no)
-			(net "Net-(R4-Pad2)")
+			(net "Net-(R7-Pad1)")
 			(pintype "passive")
 		)
@@
 			(layers "*.Cu" "*.Mask")
 			(remove_unused_layers no)
-			(net "Net-(R7-Pad2)")
+			(net "Net-(R4-Pad2)")
 			(pintype "passive")
 		)
@@
 			(layers "*.Cu" "*.Mask")
 			(remove_unused_layers no)
-			(net "Net-(R7-Pad2)")
+			(net "Net-(R7-Pad1)")
 			(pinfunction "1_1")
 			(pintype "passive")
@@
 			(layers "*.Cu" "*.Mask")
 			(remove_unused_layers no)
-			(net "Net-(U2B--)")
+			(net "Net-(C13-Pad1)")
 			(pintype "passive")
 		)
@@
 			(layers "*.Cu" "*.Mask")
 			(remove_unused_layers no)
-			(net "Net-(C13-Pad2)")
+			(net "Net-(U2B--)")
 			(pintype "passive")
 		)
@@
 			(layers "*.Cu" "*.Mask")
 			(remove_unused_layers no)
-			(net "Net-(Q3-C)")
+			(net "Net-(Q2-C)")
 			(pintype "passive")
 		)
@@
 			(layers "*.Cu" "*.Mask")
 			(remove_unused_layers no)
-			(net "Net-(U5A--)")
+			(net "KEY")
 			(pintype "passive")
 		)
@@
 			(layers "*.Cu" "*.Mask")
 			(remove_unused_layers no)
-			(net "KEY")
+			(net "Net-(U5A--)")
 			(pintype "passive")
 		)
@@
 			(layers "*.Cu" "*.Mask")
 			(remove_unused_layers no)
-			(net "Net-(U2B--)")
+			(net "Net-(C13-Pad1)")
 			(pintype "passive")
 		)
@@
 			(layers "*.Cu" "*.Mask")
 			(remove_unused_layers no)
-			(net "Net-(C13-Pad2)")
+			(net "Net-(U2B--)")
 			(pintype "passive")
 		)
@@
 			(layers "*.Cu" "*.Mask")
 			(remove_unused_layers no)
-			(net "Net-(Q5-E)")
+			(net "Net-(C10-Pad1)")
 			(pintype "passive")
 		)
@@
 			(layers "*.Cu" "*.Mask")
 			(remove_unused_layers no)
-			(net "Net-(C10-Pad2)")
+			(net "Net-(Q5-E)")
 			(pintype "passive")
 		)
@@
 			(layers "*.Cu" "*.Mask")
 			(remove_unused_layers no)
-			(net "Net-(Q3-C)")
+			(net "Net-(Q2-C)")
 			(pinfunction "C_1")
 			(pintype "passive")
@@
 			(layers "*.Cu" "*.Mask")
 			(remove_unused_layers no)
-			(net "Net-(C13-Pad2)")
+			(net "Net-(C13-Pad1)")
 			(pintype "output")
 		)

Commit message: Change switch footprints and update pcb
Parts:
- SW1: footprint Connector_PinSocket_1.00mm:PinSocket_1x06_P1.00mm_Vertical -> Connector_PinHeader_2.54mm:PinHeader_1x06_P2.54mm_Vertical
- SW2: footprint Connector_PinSocket_1.00mm:PinSocket_1x03_P1.00mm_Vertical -> Connector_PinHeader_2.54mm:PinHeader_1x03_P2.54mm_Vertical
- SW3, SW4: footprint Connector_PinSocket_1.00mm:PinSocket_1x02_P1.00mm_Vertical -> Connector_PinHeader_2.54mm:PinHeader_1x02_P2.54mm_Vertical
- moved SW4 24.7 mm to (191.2, 143.5)
- moved SW3 24.1 mm to (186.7, 143.5)
- moved SW1 21.7 mm to (178.7, 143.3)
- moved SW2 19.9 mm to (182.7, 143.5)

Commit message: Start adding pcb setup
Parts:
- moved RV2 41.7 mm to (29.6, 58.5)
- moved RV3 41.7 mm to (29.6, 72.8)
- moved RV4 41.7 mm to (29.6, 87.2)
- moved RV5 41.7 mm to (29.6, 101.5)
- moved RV6 41.7 mm to (29.6, 115.8)
Changed lines of the file:
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@@
 	)
 	(setup
+		(stackup
+			(layer "F.SilkS"
+				(type "Top Silk Screen")
+			)
+			(layer "F.Paste"
+				(type "Top Solder Paste")
+			)
+			(layer "F.Mask"
+				(type "Top Solder Mask")
+				(thickness 0.01)
+			)
+			(layer "F.Cu"
+				(type "copper")
+				(thickness 0.035)
+			)
+			(layer "dielectric 1"
+				(type "core")
+				(thickness 1.51)
+				(material "FR4")
+				(epsilon_r 4.5)
+				(loss_tangent 0.02)
+			)
+			(layer "B.Cu"
+				(type "copper")
+				(thickness 0.035)
+			)
+			(layer "B.Mask"
+				(type "Bottom Solder Mask")
+				(thickness 0.01)
+			)
+			(layer "B.Paste"
+				(type "Bottom Solder Paste")
+			)
+			(layer "B.SilkS"
+				(type "Bottom Silk Screen")
+			)
+			(copper_finish "None")
+			(dielectric_constraints no)
+		)
 		(pad_to_mask_clearance 0)
 		(allow_soldermask_bridges_in_footprints no)
@@
 		(capping no)
 		(filling no)
+		(zone_defaults)
 		(grid_origin 50.65 160)
 		(pcbplotparams
@@
 	)
 	(footprint "Cards:EDA_306"
+		(locked yes)
 		(layer "F.Cu")
 		(at 198.5 98.899)
@@
 	(footprint "Potentiometer_THT:Potentiometer_Alps_RK09K_Single_Vertical"
 		(layer "F.Cu")
-		(at 71.325 74.025)
+		(at 29.6 72.8)
 		(descr "113004U 1130A6S 11300DR 1130A8G 1130081 1130A5R 1130AP5 1130AST  D1130C3W D1130C1B D1130C3C D1130C2P Potentiometer, vertical, Alps RK09K Single, https://tech.alpsalpine.com/prod/e/pdf/potentiometer/rotarypotentiometers/rk09k/rk09k.pdf")
 		(tags "Potentiometer vertical Alps RK09K RK09D Single Snapin")
@@
 	(footprint "Potentiometer_THT:Potentiometer_Alps_RK09K_Single_Vertical"
 		(layer "F.Cu")
-		(at 71.325 88.375)
+		(at 29.6 87.15)
 		(descr "113004U 1130A6S 11300DR 1130A8G 1130081 1130A5R 1130AP5 1130AST  D1130C3W D1130C1B D1130C3C D1130C2P Potentiometer, vertical, Alps RK09K Single, https://tech.alpsalpine.com/prod/e/pdf/potentiometer/rotarypotentiometers/rk09k/rk09k.pdf")
 		(tags "Potentiometer vertical Alps RK09K RK09D Single Snapin")
@@
 	(footprint "Potentiometer_THT:Potentiometer_Alps_RK09K_Single_Vertical"
 		(layer "F.Cu")
-		(at 71.325 102.725)
+		(at 29.6 101.5)
 		(descr "113004U 1130A6S 11300DR 1130A8G 1130081 1130A5R 1130AP5 1130AST  D1130C3W D1130C1B D1130C3C D1130C2P Potentiometer, vertical, Alps RK09K Single, https://tech.alpsalpine.com/prod/e/pdf/potentiometer/rotarypotentiometers/rk09k/rk09k.pdf")
 		(tags "Potentiometer vertical Alps RK09K RK09D Single Snapin")
@@
 	(footprint "Potentiometer_THT:Potentiometer_Alps_RK09K_Single_Vertical"
 		(layer "F.Cu")
-		(at 71.325 59.675)
+		(at 29.6 58.45)
 		(descr "113004U 1130A6S 11300DR 1130A8G 1130081 1130A5R 1130AP5 1130AST  D1130C3W D1130C1B D1130C3C D1130C2P Potentiometer, vertical, Alps RK09K Single, https://tech.alpsalpine.com/prod/e/pdf/potentiometer/rotarypotentiometers/rk09k/rk09k.pdf")
 		(tags "Potentiometer vertical Alps RK09K RK09D Single Snapin")
@@
 	(footprint "Potentiometer_THT:Potentiometer_Alps_RK09K_Single_Vertical"
 		(layer "F.Cu")
-		(at 71.325 117.075)
+		(at 29.6 115.85)
 		(descr "113004U 1130A6S 11300DR 1130A8G 1130081 1130A5R 1130AP5 1130AST  D1130C3W D1130C1B D1130C3C D1130C2P Potentiometer, vertical, Alps RK09K Single, https://tech.alpsalpine.com/prod/e/pdf/potentiometer/rotarypotentiometers/rk09k/rk09k.pdf")
 		(tags "Potentiometer vertical Alps RK09K RK09D Single Snapin")
@@
 			(type solid)
 		)
+		(locked yes)
 		(layer "Edge.Cuts")
 	)
@@
 			(type solid)
 		)
+		(locked yes)
 		(layer "Edge.Cuts")
 	)
@@
 			(type solid)
 		)
+		(locked yes)
 		(layer "Edge.Cuts")
 	)
@@
 			(type solid)
 		)
+		(locked yes)
 		(layer "Edge.Cuts")
 	)
@@
 			(type solid)
 		)
+		(locked yes)
 		(layer "Edge.Cuts")
 	)
@@
 			)
 		)
+	)
+	(zone
+		(layer "F.Cu")
+		(name "Edge_1")
+		(hatch edge 0.5)
+		(connect_pads
+			(clearance 0)
+		)
+		(min_thickness 0.25)
+		(keepout
+			(tracks not_allowed)
+			(vias not_allowed)
+			(pads not_allowed)
+			(copperpour not_allowed)
+			(footprints not_allowed)
+		)
+		(placement
+			(enabled no)
+			(sheetname "/")
+		)
+		(fill
+			(thermal_gap 0.5)
+			(thermal_bridge_width 0.5)
+			(island_removal_mode 0)
+		)
+		(polygon
+			(pts
+				(xy 50.70467 57.567389) (xy 222.15467 57.567389) (xy 222.15467 55.027389) (xy 50.70467 55.027389)
+			)
+		)
+	)
+	(zone
+		(layer "F.Cu")
+		(name "Edge")
+		(hatch edge 0.5)
+		(connect_pads
+			(clearance 0)
+		)
+		(min_thickness 0.25)
+		(keepout
+			(tracks not_allowed)
+			(vias not_allowed)
+			(pads not_allowed)
+			(copperpour not_allowed)
+			(footprints not_allowed)
+		)
+		(placement
+			(enabled no)
+			(sheetname "/")
+		)
+		(fill
+			(thermal_gap 0.5)
+			(thermal_bridge_width 0.5)
+			(island_removal_mode 0)
+		)
+		(polygon
+			(pts
+				(xy 50.65 160) (xy 222.1 160) (xy 222.1 157.46) (xy 50.65 157.46)
+			)
+		)
