File: kicad_withpcb/compressor_with_pcb/compressor_with_pcb.kicad_pcb (KiCad board)
At the start: 2 copper layers, 128.3 x 105 mm, 137 parts, among them J1 EDA 306, J2 FRONT BOARD, Q1 BC549C, Q2 BC549C, Q3 BC549C, Q4 BC549C, Q5 BC549C, Q6 BC549C, Q7 BC549C, Q8 BC549C, Q9 BC549C, U1 NE5532, U2 NE5532, U3 NE5532, U4 TL072, U5 NE5532, U6 NE5532, U7 NE5532

Commit message: Split Q2's collector from the VCA tail
A wire at x = 62.23 mm joined Q2's collector (with Q8 and Q9) to the
tail node (Q3, R14, R15). They are now two nets: Net-(Q2-C) on Q2.1,
Q8.3 and Q9.3, and Net-(Q3-C) on Q3.1, R14.1 and R15.2. The board has
the new pad nets but not yet the copper to match.
Connections:
- Q3 pad 1: Net-(Q2-C) -> Net-(Q3-C)
- R14 pad 1: Net-(Q2-C) -> Net-(Q3-C)
- R15 pad 2: Net-(Q2-C) -> Net-(Q3-C)

Commit message: Re-route the tail net around R14, R15 and Q3
Two B.Cu stubs still carried Net-(Q2-C) onto the tail pads: one from the
Q8/Q9 link down to R14.1, and one from the via at (138.4, 69.8) to
R15.2. Both are gone. The existing R15.2 to Q3.1 track is now on
Net-(Q3-C), and R14.1 runs on F.Cu up between +16V and BYP_A, along
y = 73.3 to a new via at (143, 72.85), then on B.Cu to R15.2. Zones
refilled.

DRC: 0 errors, 0 unconnected, schematic parity clean (the two existing
warnings remain).
Routing:
- net Net-(Q3-C): track 0.00 -> 31.1 mm, vias 0 -> 1
- net Net-(Q2-C): track 47.5 -> 34.1 mm
