File: kicad_withpcb/compressor_with_pcb/compressor_with_pcb.kicad_pcb (KiCad board)
At the start: 2 copper layers, 128.3 x 105 mm, 137 parts, among them J1 EDA 306, J2 FRONT BOARD, Q1 BC549C, Q2 BC549C, Q3 BC549C, Q4 BC549C, Q5 BC549C, Q6 BC549C, Q7 BC549C, Q8 BC549C, Q9 BC549C, U1 NE5532, U2 NE5532, U3 NE5532, U4 TL072, U5 NE5532, U6 NE5532, U7 NE5532

Commit message: Carry the new values onto both boards' schematics and layouts
Parts:
- C10, C9: value 2u2 -> 4u7
- R21, R22: value 3k3 -> 6k8
- R35: value 20k -> 2k4
- R36: value 100k -> 200k
- R45: value 220R -> 680R
- R46: value 47R -> 150R
- R47: value 4k7 -> 12k
- R60: value 47k -> 24k
- R74: value 220k -> 1M
Changed lines of the file:
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@@
 			)
 		)
-		(property "Value" "3k3"
+		(property "Value" "6k8"
 			(at 5.08 2.37 270)
 			(layer "F.Fab")
@@
 			)
 		)
-		(property "Value" "47k"
+		(property "Value" "24k"
 			(at 5.08 2.37 90)
 			(layer "F.Fab")
@@
 			)
 		)
-		(property "Value" "47R"
+		(property "Value" "150R"
 			(at 5.08 2.37 0)
 			(layer "F.Fab")
@@
 			)
 		)
-		(property "Value" "20k"
+		(property "Value" "2k4"
 			(at 5.08 2.37 90)
 			(layer "F.Fab")
@@
 			)
 		)
-		(property "Value" "3k3"
+		(property "Value" "6k8"
 			(at 5.08 2.37 0)
 			(layer "F.Fab")
@@
 			)
 		)
-		(property "Value" "4k7"
+		(property "Value" "12k"
 			(at 5.08 2.37 0)
 			(layer "F.Fab")
@@
 			)
 		)
-		(property "Value" "220R"
+		(property "Value" "680R"
 			(at 5.08 2.37 270)
 			(layer "F.Fab")
@@
 			)
 		)
-		(property "Value" "100k"
+		(property "Value" "200k"
 			(at 5.08 2.37 90)
 			(layer "F.Fab")
@@
 			)
 		)
-		(property "Value" "220k"
+		(property "Value" "1M"
 			(at 5.08 2.37 90)
 			(layer "F.Fab")
@@
 			)
 		)
-		(property "Value" "2u2"
+		(property "Value" "4u7"
 			(at 2.5 2.5 270)
 			(layer "F.Fab")
@@
 			)
 		)
-		(property "Value" "2u2"
+		(property "Value" "4u7"
 			(at 2.5 2.5 90)
 			(layer "F.Fab")

Commit message: Retune attack and release: R45 220R, R46 47R, RV5 10k, R47 15k
The first pass ran the attack too slow (9 to 103 ms against a 2.7 to
50 ms target). Results are regenerated in the next commit.
Parts:
- R45: value 680R -> 220R
- R46: value 150R -> 47R
- R47: value 12k -> 15k
Changed lines of the file:
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@@
 			)
 		)
-		(property "Value" "150R"
+		(property "Value" "47R"
 			(at 5.08 2.37 0)
 			(layer "F.Fab")
@@
 			)
 		)
-		(property "Value" "12k"
+		(property "Value" "15k"
 			(at 5.08 2.37 0)
 			(layer "F.Fab")
@@
 			)
 		)
-		(property "Value" "680R"
+		(property "Value" "220R"
 			(at 5.08 2.37 270)
 			(layer "F.Fab")

Commit message: Stop the fast-attack overshoot: C22 47u to 4u7
C22 made STA lag STB by about 60 ms, so when CTRL-B pulled the
reference node down the steering kept moving after the control
voltage had settled, overshooting by up to 20 dB. With 4u7 the two
sides track and the overshoot is about 1 dB. RV5 back to 4k7 and RV6
to 500k, since the attack and release run slower without it.
Parts:
- C22: value 47u -> 4u7
Changed lines of the file:
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@@
 			)
 		)
-		(property "Value" "47u"
+		(property "Value" "4u7"
 			(at 1.25 4.4 0)
 			(layer "F.Fab")

Commit message: Keep R74 at 220k and write up the new results
R74 at 1M only moved CTRL-B's resting offset further from zero with an
NE5532 in U4, so it goes back to 220k. The sim README now lists the
eleven changed values with before, after and target figures.
Parts:
- R74: value 1M -> 220k
Changed lines of the file:
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@@
 			)
 		)
-		(property "Value" "1M"
+		(property "Value" "220k"
 			(at 5.08 2.37 90)
 			(layer "F.Fab")

Commit message: Use 100k pots for RV3 and RV6, and steady the sidechain high-pass
RK09K pots stop at 100k. RV3 becomes 100kA with R35 1k and R36 82k,
which scales the threshold network and keeps the -20 to +20 dBu range.
RV6 becomes 100k, so the slowest release drops to about 0.4 s.

R35 at 2k4 had also loaded the sidechain high-pass (C14 into R38), so at
the lowest threshold its corner rose to about 400 Hz. R38 1k and C14 2u2
hold it between about 80 and 160 Hz across the threshold knob.
Parts:
- C14: value 220n -> 2u2
- R35: value 2k4 -> 1k
- R36: value 200k -> 82k
- R38: value 10k -> 1k
Changed lines of the file:
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@@
 			)
 		)
-		(property "Value" "2k4"
+		(property "Value" "1k"
 			(at 5.08 2.37 90)
 			(layer "F.Fab")
@@
 			)
 		)
-		(property "Value" "10k"
+		(property "Value" "1k"
 			(at 5.08 2.37 270)
 			(layer "F.Fab")
@@
 			)
 		)
-		(property "Value" "220n"
+		(property "Value" "2u2"
 			(at 2.5 2.5 90)
 			(layer "F.Fab")
@@
 			)
 		)
-		(property "Value" "200k"
+		(property "Value" "82k"
 			(at 5.08 2.37 90)
 			(layer "F.Fab")

Commit message: Fit real film capacitors on the main board and use Altronics pots for RV5/RV6
RV5 (ATTACK) goes 4k7 -> 10k and RV6 (RELEASE) 500k -> 1M, the nearest
Altronics 9 mm values (R1946, R1950), on the split sheets, both boards
and design.py; the Sim.Params follow (R=10000, R=1e+06).

C5, C8, C9, C10, C14, C15 and C35 were drawn as 7 x 2.5 mm on 5 mm, which
no 2.2-10 uF film part fits. They now use stock KiCad footprints for
in-stock element14 parts:
  10 uF  C5 C8 C15  TDK B32562H1106K000   C_Rect_L16.5mm_W11.8mm_P15.00mm_MKT
  4.7 uF C9 C10     TDK B32562H1475K000   C_Rect_L16.5mm_W7.3mm_P15.00mm_MKT
  2.2 uF C14 C35    KEMET MMK5225K63J06L4 C_Rect_L7.2mm_W7.2mm_P5.00mm_FKS2...

To make room, small parts were re-placed by script (the caps near their
old spots, displaced parts re-homed, then same-footprint parts swapped to
cut wire length; transistors, ICs, connectors and trimmers did not move)
and the main board was re-routed with Freerouting, keeping the original
card-finger stubs. DRC 0 errors, 0 unconnected, schematic parity clean;
ERC 0 errors. The BOM names the element14 parts.
Parts:
- C10, C9: footprint Capacitor_THT:C_Rect_L7.0mm_W2.5mm_P5.00mm -> Capacitor_THT:C_Rect_L16.5mm_W7.3mm_P15.00mm_MKT
- C14, C35: footprint Capacitor_THT:C_Rect_L7.0mm_W2.5mm_P5.00mm -> Capacitor_THT:C_Rect_L7.2mm_W7.2mm_P5.00mm_FKS2_FKP2_MKS2_MKP2
- C15, C5, C8: footprint Capacitor_THT:C_Rect_L7.0mm_W2.5mm_P5.00mm -> Capacitor_THT:C_Rect_L16.5mm_W11.8mm_P15.00mm_MKT
- moved R28 83.8 mm to (87.5, 69.0), turned to -90 degrees
- moved C19 73.7 mm to (144.0, 74.6), turned to 0 degrees
- moved R10 53.4 mm to (171.0, 142.5)
- moved R24 49.6 mm to (168.6, 105.4), turned to 90 degrees
- moved R9 49.0 mm to (156.0, 137.4), turned to 90 degrees
- moved LED1 44.3 mm to (118.7, 135.7), turned to 180 degrees
- moved R22 42.7 mm to (155.9, 116.3), turned to 0 degrees
- moved R26 40.8 mm to (126.0, 85.1)
- moved C7 39.8 mm to (170.1, 108.4), turned to 180 degrees
- moved R23 39.6 mm to (129.2, 109.2), turned to -90 degrees
- moved R38 35.8 mm to (119.0, 108.0)
- moved R17 35.0 mm to (185.5, 88.2)
- moved R7 32.1 mm to (152.6, 120.5), turned to -90 degrees
- moved C11 29.9 mm to (129.4, 102.9)
- moved R12 29.1 mm to (158.5, 89.2), turned to 0 degrees
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Routing:
- net VBIAS: track 32.9 -> 147.4 mm
- net BYP_A: track 92.4 -> 16.8 mm, vias 4 -> 0
- net HPF_B: track 125.2 -> 64.4 mm, vias 2 -> 0
- net LINK: track 197.0 -> 141.2 mm, vias 5 -> 4
- net Net-(Q5-B): track 16.2 -> 67.2 mm, vias 0 -> 1
- net Net-(U1B-+): track 64.3 -> 15.9 mm, vias 1 -> 0
- net KEY: track 160.5 -> 112.3 mm, vias 1 -> 0
- net Net-(LED1-A): track 52.3 -> 5.11 mm, vias 3 -> 0
- net AGND: track 678.7 -> 719.5 mm, vias 1 -> 5
- net CTRL-B: track 60.0 -> 95.8 mm, vias 0 -> 1
- net RATIO_CW: track 61.5 -> 26.4 mm, vias 2 -> 1
- net Net-(U6A-+): track 18.2 -> 49.6 mm
- net Net-(D7-K): track 6.67 -> 36.5 mm, vias 0 -> 2
- net Net-(R86-Pad1): track 42.5 -> 14.9 mm
- net OUT+: track 165.2 -> 138.2 mm, vias 4 -> 1
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