File: kicad_withpcb/compressor_with_pcb/compressor_with_pcb.kicad_sch (KiCad schematic)
At the start: 90 parts, among them J1 EDA 306, Q1 BC549C, Q2 BC549C, Q3 BC549C, Q4 BC549C, Q5 BC549C, Q6 BC549C, Q7 BC549C, Q8 BC549C, Q9 BC549C, SW1 BYPASS, SW2 INT/EXT, SW3 HPF DEFEAT, SW4 LINK, U1 NE5532, U2 NE5532, U3 NE5532, U4 NE5532, U5 NE5532, U6 NE5532

Commit message: Add power shtuff and meters to big boy schematic
Parts:
- added C16, C17, C6: 100u, Capacitor_THT:CP_Radial_D6.3mm_P2.50mm, symbol Device:C_Polarized
- added C18: 10n, Capacitor_THT:C_Disc_D5.0mm_W2.5mm_P5.00mm, symbol Device:C
- added C19, C21, C22, C38: 47u, Capacitor_THT:CP_Radial_D6.3mm_P2.50mm, symbol Device:C_Polarized
- added C20, C23, C24, C25, C26, C27, C28, C29, C30, C31, C32, C33, C34, C36, C37, C39, C40, C7: 100n, Capacitor_THT:C_Disc_D5.0mm_W2.5mm_P5.00mm, symbol Device:C
- added C35: 2u2, Capacitor_THT:C_Rect_L7.0mm_W2.5mm_P5.00mm, symbol Device:C
- added D10: BZX79-C5V1, Diode_THT:D_DO-35_SOD27_P7.62mm_Horizontal, symbol Device:D_Zener
- added D11, D12: 1N4148, Diode_THT:D_DO-35_SOD27_P7.62mm_Horizontal, symbol Device:D
- added D20, D21, D22, D23, D24, D25, D26, D30, D31, D32, D33, D34, D35, D36: meter, LED_THT:LED_D2.0mm_W4.0mm_H2.8mm_FlatTop, symbol Device:LED
- added D8, D9: 1N4004, Diode_THT:D_DO-41_SOD81_P7.62mm_Horizontal, symbol Device:D
- added LED1: GR, LED_THT:LED_D3.0mm, symbol Device:LED
- added R10: 11k, Resistor_THT:R_Axial_DIN0207_L6.3mm_D2.5mm_P10.16mm_Horizontal, symbol Device:R
- added R48: 0R, Resistor_THT:R_Axial_DIN0207_L6.3mm_D2.5mm_P10.16mm_Horizontal, symbol Device:R
- added R50, R51: 10R, Resistor_THT:R_Axial_DIN0207_L6.3mm_D2.5mm_P10.16mm_Horizontal, symbol Device:R
- added R52: 100R, Resistor_THT:R_Axial_DIN0207_L6.3mm_D2.5mm_P10.16mm_Horizontal, symbol Device:R
- added R53: 1k8, Resistor_THT:R_Axial_DIN0207_L6.3mm_D2.5mm_P10.16mm_Horizontal, symbol Device:R
- added R60: 47k, Resistor_THT:R_Axial_DIN0207_L6.3mm_D2.5mm_P10.16mm_Horizontal, symbol Device:R
- added R61: 1k33, Resistor_THT:R_Axial_DIN0207_L6.3mm_D2.5mm_P10.16mm_Horizontal, symbol Device:R
- added R62: 23k2, Resistor_THT:R_Axial_DIN0207_L6.3mm_D2.5mm_P10.16mm_Horizontal, symbol Device:R
- added R68, R87: 1k, Resistor_THT:R_Axial_DIN0207_L6.3mm_D2.5mm_P10.16mm_Horizontal, symbol Device:R
- added R69: 36k, Resistor_THT:R_Axial_DIN0207_L6.3mm_D2.5mm_P10.16mm_Horizontal, symbol Device:R
- added R77: 3k9, Resistor_THT:R_Axial_DIN0207_L6.3mm_D2.5mm_P10.16mm_Horizontal, symbol Device:R
- added R84, R85, R86, R94: 10k, Resistor_THT:R_Axial_DIN0207_L6.3mm_D2.5mm_P10.16mm_Horizontal, symbol Device:R
- added R88: 100k, Resistor_THT:R_Axial_DIN0207_L6.3mm_D2.5mm_P10.16mm_Horizontal, symbol Device:R
- added R89, R91: 2k7, Resistor_THT:R_Axial_DIN0207_L6.3mm_D2.5mm_P10.16mm_Horizontal, symbol Device:R
- added R9: 68k, Resistor_THT:R_Axial_DIN0207_L6.3mm_D2.5mm_P10.16mm_Horizontal, symbol Device:R
- added R90, R92: 8k2, Resistor_THT:R_Axial_DIN0207_L6.3mm_D2.5mm_P10.16mm_Horizontal, symbol Device:R
- added R93: 18k, Resistor_THT:R_Axial_DIN0207_L6.3mm_D2.5mm_P10.16mm_Horizontal, symbol Device:R
- added RV7, RV8: 20k, Potentiometer_THT:Potentiometer_Bourns_3296W_Vertical, symbol Device:R_Potentiometer
- added unit 3 of U1
- added U10: LM3915, Package_DIP:DIP-18_W7.62mm, symbol Driver_LED:LM3914N
- added unit 3 of U2
- added unit 3 of U3
- added unit 3 of U5
- added unit 3 of U6
- added U7, U8: NE5532, Package_DIP:DIP-8_W7.62mm, symbol Amplifier_Operational:NE5532
- added U9: LM3914, Package_DIP:DIP-18_W7.62mm, symbol Driver_LED:LM3914N
- U4: value NE5532 -> TL072
Connections:
- net +IN+4 is gone; now on net IN+: J1.10 (Pin_10), R6.1
- net +IN-2 is gone; now on net AUXIN-: J1.9 (Pin_9)
- net +OUT+4 is gone; now on net OUT+: J1.2 (Pin_2)
- net +OUT-2 is gone; now on net AUXOUT+: J1.3 (Pin_3)
- net -IN-2 is gone; now on net AUXOUT-: J1.7 (Pin_7)
- net -OUT is gone; now on net OUT-: J1.4 (Pin_4)
- net GAIN_ADJ is gone; now on net AUXIN+: J1.11 (Pin_11)
- net SC_LINK is gone; now on net LINK: J1.6 (Pin_6)
- net +16V: now also C16.1, C23.1, C24.1, C25.1, C26.1, C27.1, C28.1, C36.1, C37.1, C38.1, C39.1, D20.2 (A), D21.2 (A), D22.2 (A), D23.2 (A), D24.2 (A), D25.2 (A), D26.2 (A), D30.2 (A), D31.2 (A), D32.2 (A), D33.2 (A), D34.2 (A), D35.2 (A), D36.2 (A), D8.1 (K), R50.2, R60.1, R9.1, U1.8 (V+), U10.3 (V+), U2.8 (V+), U3.8 (V+), U5.8 (V+), U6.8 (V+), U7.8 (V+), U8.8 (V+), U9.3 (V+); no longer J1.12 (Pin_12)
- net -16V: now also C17.2, C29.1, C30.1, C31.1, C32.1, C33.1, C34.1, C40.1, D9.2 (A), R51.2, R53.1, U1.4 (V-), U2.4 (V-), U3.4 (V-), U5.4 (V-), U6.4 (V-), U7.4 (V-), U8.4 (V-); no longer J1.14 (Pin_14)
- net -5V1: now also C19.2, C20.1, D10.2 (A), R53.2
- net AGND: now also C16.2, C17.1, C18.2, C19.1, C20.2, C21.2, C22.2, C23.2, C24.2, C25.2, C26.2, C27.2, C28.2, C29.2, C30.2, C31.2, C32.2, C33.2, C34.2, C35.2, C36.2, C37.2, C38.2, C39.2, C40.2, C6.2, C7.2, D10.1 (K), D12.2 (A), D8.2 (A), D9.1 (K), R10.2, R48.2, R52.2, R62.2, R77.1, R85.2, R88.2, R90.2, R92.2, RV8.3, U10.2 (V-), U10.4 (RLO), U9.2 (V-), U9.4 (RLO); no longer J1.5 (Pin_5)
- net CHASSIS: now also C18.1, R52.1; no longer J1.1 (Pin_1)
- net CTRL-B: now also LED1.1 (K), R69.2, R84.1
- net GND: now also J1.5 (Pin_5); no longer J1.13 (Pin_13)
- net IN+: now also R5.1
- net IN-: now also J1.8 (Pin_8)
- net OUT-A: now also RV8.1
- net PAD: no longer R8.1, RV1.2, RV1.3
- net STA: now also U7.1, U7.2 (-)
- net STB: now also R68.2, R69.1
- net VBIAS: now also C6.1, C7.1, R10.1, R9.2
- net +48V renamed +48V-IN
- removed net -IN+4: J1.8 (Pin_8), R5.1
- new net: D24.1 (K), U9.15 (LED5)
- new net: R85.1, U8.5 (+)
- new net: R84.2, R93.2, RV7.1, U8.6 (-)
- new net: R94.1, RV7.2, RV7.3, U8.7
- new net: D20.1 (K), U9.1 (LED1)
- new net: D26.1 (K), U9.13 (LED7)
- new net: D25.1 (K), U9.14 (LED6)
- new net: D23.1 (K), U9.16 (LED4)
- new net: D22.1 (K), U9.17 (LED3)
- new net: D21.1 (K), U9.18 (LED2)
- new net: D12.1 (K), R94.2, U9.5 (SIG)
- new net: R89.1, R93.1, U9.6 (RHI), U9.7 (REFOUT)
- new net: R89.2, R90.1, U9.8 (REFADJ)
- new net: R87.1, U8.1
- new net: D11.2 (A), R87.2
- new net: D30.1 (K), U10.16 (LED4)
- new net: C22.1, R61.2, R62.1, U7.3 (+)
- new net: R86.1, RV8.2
- new net: R86.2, U8.3 (+)
- new net: C35.1, D11.1 (K), R88.1, U10.5 (SIG), U8.2 (-)
- new net: LED1.2 (A), R77.2
- new net: D32.1 (K), U10.14 (LED6)
- new net: R91.2, R92.1, U10.8 (REFADJ)
- new net: D35.1 (K), U10.11 (LED9)
- new net: D36.1 (K), U10.10 (LED10)
- new net: C21.1, R60.2, R61.1, R68.1
- new net: D34.1 (K), U10.12 (LED8)
- new net: D33.1 (K), U10.13 (LED7)
- new net: R91.1, U10.6 (RHI), U10.7 (REFOUT)
- new net: R8.1, RV1.2, RV1.3
- new net: D31.1 (K), U10.15 (LED5)
- new net +16V-IN: J1.12 (Pin_12), R50.1
- new net -16V-IN: J1.14 (Pin_14), R51.1
- new net CHASSIS_GND: J1.1 (Pin_1)
- new net Earth: J1.13 (Pin_13)
- new net PGND: R48.1
- no-connect marks 0 -> 8
Other:
- note added: "+16 V RAIL ENTRY"
- note added: "-16 V RAIL ENTRY"
- note added: "-5V1 REFERENCE"
- note added: "CELL BIAS"
- note added: "GAIN-REDUCTION METER"
- note added: "GROUNDING"
- note added: "OP-AMP SUPPLY DECOUPLING"
- note added: "On board copper female connector. 15 Poles. Labeling from Midas."
- note added: "STEERING REFERENCE"
- note removed: "On board copper female connector. 15 Poles. Labeling from RADIAL."
- moved on the sheet: R28, R32, R33, R34, R8, R80, R81, R82, R83, SW1A, SW1B, U5A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

Commit message: Cleanup meters & power in schematic
Parts:
- removed C39, C40: 100n, Capacitor_THT:C_Disc_D5.0mm_W2.5mm_P5.00mm, symbol Device:C
- removed unit 3 of U8
- added C41, C42: 100n, Capacitor_THT:C_Disc_D5.0mm_W2.5mm_P5.00mm, symbol Device:C
- added unit 3 of U7
- U10: value LM3915 -> LM3914
- renumbered U5 to U4, U6 to U5, U7 to U6, U8 to U7
Connections:
- net +16V: now also R9.2, C41.1, U7.8 (V+); no longer R9.1
- net -16V: now also C42.1, U7.4 (V-)
- net AGND: now also C41.2, C42.2
- net VBIAS: now also R9.1; no longer R9.2
- net at U7.5 (+): now also R86.2; no longer R85.1
- net at R84.2, R93.2, RV7.1: now also U7.2 (-); no longer U7.6 (-)
- net at RV7.2, RV7.3: now also R94.2, U7.1; no longer R94.1, U7.7
- net at D12.1 (K), U9.5 (SIG): now also R94.1; no longer R94.2
- net at R87.1: now also D11.2 (A); no longer U7.1
- net at R87.2: now also U7.7; no longer D11.2 (A)
- net at U7.3 (+): now also R85.1; no longer R86.2
- net at C35.1, D11.1 (K), R88.1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: now also U7.6 (-); no longer U7.2 (-)
- net at R92.1, U10.8 (REFADJ): now also R91.1; no longer R91.2
- net at U10.6 (RHI), U10.7 (REFOUT): now also R91.2; no longer R91.1
- no-connect marks 8 -> 5
Other:
- note added: "+16 V RAIL"
- note added: "-16 V RAIL"
- note added: "-5V1 CREATION"
- note added: "GAIN RED. METER"
- note added: "OP-AMP POWER DECOUPLING"
- note added: "PWR FLAGs"
- note removed: "+16 V RAIL ENTRY"
- note removed: "-16 V RAIL ENTRY"
- note removed: "-5V1 REFERENCE"
- note removed: "GAIN-REDUCTION METER"
- note removed: "OP-AMP SUPPLY DECOUPLING"
- moved on the sheet: C13, C14, C15, C16, C17, C18, C19, C20, C21, C22, C23, C24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

Commit message: Fix issues with schematic and basic add pcb
Parts:
- U10: value LM3914 -> LM3915
- U4: value NE5532 -> TL072
Connections:
- net CHASSIS_GND is gone; now on net CHASSIS: J1.1 (Pin_1)
- net Earth is gone; now on net PGND: J1.13 (Pin_13)
- net GND is gone; now on net AGND: J1.5 (Pin_5)
- net IN+: no longer R5.1
- net IN-: now also R5.1
- net PAD: now also R8.1, RV1.2, RV1.3
Changed lines of the file:
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@@
 	)
 	(junction
+		(at 107.95 62.23)
+		(diameter 0)
+		(color 0 0 0 0)
+	)
+	(junction
 		(at 382.27 93.98)
 		(diameter 0)
@@
 	(wire
 		(pts
+			(xy 111.76 62.23) (xy 107.95 62.23)
+		)
+		(stroke
+			(width 0)
+			(type default)
+		)
+	)
+	(wire
+		(pts
 			(xy 198.12 113.03) (xy 198.12 106.68)
 		)
@@
 	(wire
 		(pts
-			(xy 35.56 85.09) (xy 35.56 87.63)
+			(xy 35.56 85.09) (xy 35.56 88.9)
 		)
 		(stroke
@@
 	(wire
 		(pts
-			(xy 107.95 58.42) (xy 107.95 64.77)
+			(xy 107.95 58.42) (xy 107.95 62.23)
 		)
 		(stroke
@@
 	(wire
 		(pts
+			(xy 107.95 62.23) (xy 107.95 64.77)
+		)
+		(stroke
+			(width 0)
+			(type default)
+		)
+	)
+	(wire
+		(pts
 			(xy 354.33 207.01) (xy 374.65 207.01)
 		)
@@
 		)
 	)
-	(global_label "CHASSIS_GND"
+	(global_label "CHASSIS"
 		(shape bidirectional)
 		(at 381 15.24 180)
@@
 		)
 	)
+	(global_label "PAD"
+		(shape bidirectional)
+		(at 111.76 62.23 0)
+		(effects
+			(font
+				(size 1.27 1.27)
+			)
+			(justify left)
+		)
+		(property "Intersheetrefs" "${INTERSHEET_REFS}"
+			(at 111.76 62.23 0)
+			(hide yes)
+			(show_name no)
+			(do_not_autoplace no)
+			(effects
+				(font
+					(size 1.27 1.27)
+				)
+			)
+		)
+	)
 	(global_label "IN+"
 		(shape bidirectional)
@@
 		)
 	)
-	(global_label "IN+"
+	(global_label "IN-"
 		(shape bidirectional)
-		(at 35.56 87.63 270)
+		(at 35.56 88.9 270)
 		(effects
 			(font
@@
 		)
 		(property "Intersheetrefs" "${INTERSHEET_REFS}"
-			(at 35.56 87.63 90)
+			(at 35.56 88.9 90)
 			(hide yes)
 			(show_name no)
@@
 			)
 		)
-		(property "Value" "GND"
+		(property "Value" "AGND"
 			(at 368.9858 25.527 0)
 			(show_name no)
@@
 			)
 		)
-		(property "Value" "Earth"
+		(property "Value" "PGND"
 			(at 369.062 48.26 0)
 			(show_name no)
@@
 			)
 		)
-		(property "Value" "NE5532"
+		(property "Value" "TL072"
 			(at 109.474 261.62 90)
 			(show_name no)
@@
 		(dnp no)
 		(property "Reference" "R5"
-			(at 31.75 82.55 0)
+			(at 37.084 84.582 90)
 			(show_name no)
 			(do_not_autoplace no)
@@
 		)
 		(property "Value" "100R"
-			(at 31.75 79.38 0)
+			(at 34.544 84.074 90)
 			(show_name no)
 			(do_not_autoplace no)
@@
 			)
 		)
-		(property "Value" "LM3914"
+		(property "Value" "LM3915"
 			(at 437.896 107.696 0)
 			(show_name no)

Commit message: Add last few footprints for switches as header pins
Parts:
- SW1: footprint (none) -> Connector_PinSocket_1.00mm:PinSocket_1x06_P1.00mm_Vertical
- SW2: footprint (none) -> Connector_PinSocket_1.00mm:PinSocket_1x03_P1.00mm_Vertical
- SW3, SW4: footprint (none) -> Connector_PinSocket_1.00mm:PinSocket_1x02_P1.00mm_Vertical
Changed lines of the file:
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@@
 			)
 		)
-		(property "Footprint" ""
+		(property "Footprint" "Connector_PinSocket_1.00mm:PinSocket_1x02_P1.00mm_Vertical"
 			(at 139.7 180.34 0)
 			(hide yes)
@@
 			)
 		)
-		(property "Footprint" ""
+		(property "Footprint" "Connector_PinSocket_1.00mm:PinSocket_1x02_P1.00mm_Vertical"
 			(at 57.15 119.38 0)
 			(hide yes)
@@
 			)
 		)
-		(property "Footprint" ""
+		(property "Footprint" "Connector_PinSocket_1.00mm:PinSocket_1x03_P1.00mm_Vertical"
 			(at 21.59 137.16 0)
 			(hide yes)
@@
 			)
 		)
-		(property "Footprint" ""
+		(property "Footprint" "Connector_PinSocket_1.00mm:PinSocket_1x06_P1.00mm_Vertical"
 			(at 370.84 228.6 0)
 			(hide yes)
@@
 			)
 		)
-		(property "Footprint" ""
+		(property "Footprint" "Connector_PinSocket_1.00mm:PinSocket_1x06_P1.00mm_Vertical"
 			(at 401.32 214.63 0)
 			(hide yes)

Commit message: Finish Schematic re-organisation and begin pcb
Connections:
- net KEY: now also R82.1; no longer R82.2
- net at Q3.1 (C), R15.2: now also Q2.1 (C), Q8.3 (E), Q9.3 (E), R14.1; no longer R14.2
- net at Q5.3 (E), R20.1: now also C10.2; no longer C10.1
- net at C13.1, R30.1: now also R32.1, U2.7; no longer R29.2, U2.6 (-)
- net at C13.2, R30.2: now also R29.2, U2.6 (-); no longer R32.1, U2.7
- net at R22.1: now also C10.1; no longer C10.2
- net at R80.2, U5.2 (-): now also R82.2; no longer R82.1
- net at Q1.3 (E): now also R14.2; no longer R14.1
- net at R4.2, U1.1: now also R7.2; no longer R7.1
- net at RV1.1: now also R7.1; no longer R7.2
Other:
- note added: "Aux Output & Input Setup"
- note added: "Input Level Meter & Gain Reduction Meter"
- note added: "Input Section Buffer and Unbalance the Input Before Sending it to the Pad"
- note added: "Output Chain, Buffer Op=Amps and Signal Balancing"
- note added: "Sidechain, Threshold, Ratio, Attack & Release Control"
- note added: "The Gain Cell Nine Transistors & an Op=Amp to act as a Voltage Controlled Amplifier"
- moved on the sheet: C1, C10, C11, C13, C14, C15, C2, C21, C22, C3, C35, C36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

Commit message: Change switch footprints and update pcb
Parts:
- SW1: footprint Connector_PinSocket_1.00mm:PinSocket_1x06_P1.00mm_Vertical -> Connector_PinHeader_2.54mm:PinHeader_1x06_P2.54mm_Vertical
- SW2: footprint Connector_PinSocket_1.00mm:PinSocket_1x03_P1.00mm_Vertical -> Connector_PinHeader_2.54mm:PinHeader_1x03_P2.54mm_Vertical
- SW3, SW4: footprint Connector_PinSocket_1.00mm:PinSocket_1x02_P1.00mm_Vertical -> Connector_PinHeader_2.54mm:PinHeader_1x02_P2.54mm_Vertical
Changed lines of the file:
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@@
 			)
 		)
-		(property "Footprint" "Connector_PinSocket_1.00mm:PinSocket_1x02_P1.00mm_Vertical"
-			(at 88.9 184.15 0)
+		(property "Footprint" "Connector_PinHeader_2.54mm:PinHeader_1x02_P2.54mm_Vertical"
+			(at 96.012 193.04 0)
 			(hide yes)
 			(show_name no)
@@
 			)
 		)
-		(property "Footprint" "Connector_PinSocket_1.00mm:PinSocket_1x02_P1.00mm_Vertical"
+		(property "Footprint" "Connector_PinHeader_2.54mm:PinHeader_1x02_P2.54mm_Vertical"
 			(at 57.15 123.19 0)
 			(hide yes)
@@
 			)
 		)
-		(property "Footprint" "Connector_PinSocket_1.00mm:PinSocket_1x03_P1.00mm_Vertical"
+		(property "Footprint" "Connector_PinHeader_2.54mm:PinHeader_1x03_P2.54mm_Vertical"
 			(at 21.59 140.97 0)
 			(hide yes)
@@
 			)
 		)
-		(property "Footprint" "Connector_PinSocket_1.00mm:PinSocket_1x06_P1.00mm_Vertical"
+		(property "Footprint" "Connector_PinHeader_2.54mm:PinHeader_1x06_P2.54mm_Vertical"
 			(at 269.24 276.86 0)
 			(hide yes)
@@
 			)
 		)
-		(property "Footprint" "Connector_PinSocket_1.00mm:PinSocket_1x06_P1.00mm_Vertical"
+		(property "Footprint" "Connector_PinHeader_2.54mm:PinHeader_1x06_P2.54mm_Vertical"
 			(at 314.96 240.03 0)
 			(hide yes)

Commit message: Start adding pcb setup
Connections:
- no-connect marks 5 -> 8
Other:
- note added: "Output Chain, Buffer Op-Amps and Signal Balancing"
- note added: "The Gain Cell Nine Transistors & an Op-Amp to act as a Voltage Controlled Amplifier"
- note removed: "Output Chain, Buffer Op=Amps and Signal Balancing"
- note removed: "The Gain Cell Nine Transistors & an Op=Amp to act as a Voltage Controlled Amplifier"
Changed lines of the file:
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@@
 		)
 	)
-	(text "Output Chain, Buffer Op=Amps and Signal Balancing"
+	(text "Output Chain, Buffer Op-Amps and Signal Balancing"
 		(exclude_from_sim no)
 		(at 226.06 227.584 0)
@@
 		)
 	)
-	(text "The Gain Cell\nNine Transistors & an Op=Amp to act as a Voltage Controlled Amplifier\n"
+	(text "The Gain Cell\nNine Transistors & an Op-Amp to act as a Voltage Controlled Amplifier\n"
 		(exclude_from_sim no)
 		(at 13.97 20.574 0)
@@
 	)
 	(junction
+		(at 25.4 62.23)
+		(diameter 0)
+		(color 0 0 0 0)
+	)
+	(junction
 		(at 344.17 127)
 		(diameter 0)
@@
 	)
 	(no_connect
+		(at 373.38 143.51)
+	)
+	(no_connect
+		(at 373.38 140.97)
+	)
+	(no_connect
 		(at 295.91 163.83)
 	)
 	(no_connect
+		(at 373.38 146.05)
+	)
+	(no_connect
 		(at 316.23 158.75)
 	)
@@
 	(wire
 		(pts
+			(xy 25.4 55.88) (xy 25.4 62.23)
+		)
+		(stroke
+			(width 0)
+			(type default)
+		)
+	)
+	(wire
+		(pts
 			(xy 40.64 48.26) (xy 38.1 48.26)
 		)
@@
 	(wire
 		(pts
+			(xy 25.4 55.88) (xy 39.37 55.88)
+		)
+		(stroke
+			(width 0)
+			(type default)
+		)
+	)
+	(wire
+		(pts
 			(xy 198.12 151.13) (xy 198.12 162.56)
 		)
@@
 	(wire
 		(pts
-			(xy 39.37 55.88) (xy 35.56 55.88)
-		)
-		(stroke
-			(width 0)
-			(type default)
-		)
-	)
-	(wire
-		(pts
 			(xy 293.37 130.81) (xy 293.37 128.27)
 		)
@@
 		)
 	)
-	(global_label "VBIAS"
-		(shape bidirectional)
-		(at 35.56 55.88 180)
-		(effects
-			(font
-				(size 1.27 1.27)
-			)
-			(justify right)
-		)
-		(property "Intersheetrefs" "${INTERSHEET_REFS}"
-			(at 35.56 55.88 0)
-			(hide yes)
-			(show_name no)
-			(do_not_autoplace no)
-			(effects
-				(font
-					(size 1.27 1.27)
-				)
-			)
-		)
-	)
 	(global_label "KEY"
 		(shape bidirectional)
@@
 		)
 		(property "Value" "PGND"
-			(at 369.062 48.26 0)
+			(at 368.046 48.26 0)
 			(show_name no)
 			(do_not_autoplace no)
