File: kicad_withpcb/compressor_with_pcb/compressor_with_pcb.kicad_sch (KiCad schematic)
At the start: 167 parts, among them J1 EDA 306, J2 FRONT BOARD, Q1 BC549C, Q2 BC549C, Q3 BC549C, Q4 BC549C, Q5 BC549C, Q6 BC549C, Q7 BC549C, Q8 BC549C, Q9 BC549C, SW1 BYPASS, SW2 INT/EXT, SW3 HPF DEFEAT, SW4 LINK, U1 NE5532, U10 LM3915, U2 NE5532, U3 NE5532, U4 TL072, U5 NE5532, U6 NE5532, U7 NE5532, U9 LM3914

Commit message: Keep R74 at 220k and write up the new results
R74 at 1M only moved CTRL-B's resting offset further from zero with an
NE5532 in U4, so it goes back to 220k. The sim README now lists the
eleven changed values with before, after and target figures.
Parts:
- R74: value 1M -> 220k
Changed lines of the file:
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@@
 			)
 		)
-		(property "Value" "1M"
+		(property "Value" "220k"
 			(at 81.534 152.4 90)
 			(show_name no)

Commit message: Use 100k pots for RV3 and RV6, and steady the sidechain high-pass
RK09K pots stop at 100k. RV3 becomes 100kA with R35 1k and R36 82k,
which scales the threshold network and keeps the -20 to +20 dBu range.
RV6 becomes 100k, so the slowest release drops to about 0.4 s.

R35 at 2k4 had also loaded the sidechain high-pass (C14 into R38), so at
the lowest threshold its corner rose to about 400 Hz. R38 1k and C14 2u2
hold it between about 80 and 160 Hz across the threshold knob.
Parts:
- C14: value 220n -> 2u2
- R35: value 2k4 -> 1k
- R36: value 200k -> 82k
- R38: value 10k -> 1k
- RV3: value 250kA -> 100kA
- RV6: value 500k -> 100k
Changed lines of the file:
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@@
 			)
 		)
-		(property "Value" "500k"
+		(property "Value" "100k"
 			(at 140.97 180.34 90)
 			(show_name no)
@@
 			)
 		)
-		(property "Value" "2k4"
+		(property "Value" "1k"
 			(at 85.09 128.016 90)
 			(show_name no)
@@
 			)
 		)
-		(property "Value" "200k"
+		(property "Value" "82k"
 			(at 108.204 130.81 90)
 			(show_name no)
@@
 			)
 		)
-		(property "Value" "10k"
+		(property "Value" "1k"
 			(at 64.516 136.398 90)
 			(show_name no)
@@
 			)
 		)
-		(property "Value" "250kA"
+		(property "Value" "100kA"
 			(at 72.136 122.682 90)
 			(show_name no)
@@
 			)
 		)
-		(property "Value" "220n"
+		(property "Value" "2u2"
 			(at 53.34 129.54 90)
 			(show_name no)

Commit message: Put RV6 back to 500k, to be a Bourns PTV09
RK09K stops at 100k, which would cut the slowest release to about 0.4 s.
Lyn chose a 500k Bourns PTV09 instead, keeping it near 1.8 s.
Parts:
- RV6: value 100k -> 500k
Changed lines of the file:
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@@
 			)
 		)
-		(property "Value" "100k"
+		(property "Value" "500k"
 			(at 140.97 180.34 90)
 			(show_name no)

Commit message: Fit real film capacitors on the main board and use Altronics pots for RV5/RV6
RV5 (ATTACK) goes 4k7 -> 10k and RV6 (RELEASE) 500k -> 1M, the nearest
Altronics 9 mm values (R1946, R1950), on the split sheets, both boards
and design.py; the Sim.Params follow (R=10000, R=1e+06).

C5, C8, C9, C10, C14, C15 and C35 were drawn as 7 x 2.5 mm on 5 mm, which
no 2.2-10 uF film part fits. They now use stock KiCad footprints for
in-stock element14 parts:
  10 uF  C5 C8 C15  TDK B32562H1106K000   C_Rect_L16.5mm_W11.8mm_P15.00mm_MKT
  4.7 uF C9 C10     TDK B32562H1475K000   C_Rect_L16.5mm_W7.3mm_P15.00mm_MKT
  2.2 uF C14 C35    KEMET MMK5225K63J06L4 C_Rect_L7.2mm_W7.2mm_P5.00mm_FKS2...

To make room, small parts were re-placed by script (the caps near their
old spots, displaced parts re-homed, then same-footprint parts swapped to
cut wire length; transistors, ICs, connectors and trimmers did not move)
and the main board was re-routed with Freerouting, keeping the original
card-finger stubs. DRC 0 errors, 0 unconnected, schematic parity clean;
ERC 0 errors. The BOM names the element14 parts.
Parts:
- C10, C9: footprint Capacitor_THT:C_Rect_L7.0mm_W2.5mm_P5.00mm -> Capacitor_THT:C_Rect_L16.5mm_W7.3mm_P15.00mm_MKT
- C14, C35: footprint Capacitor_THT:C_Rect_L7.0mm_W2.5mm_P5.00mm -> Capacitor_THT:C_Rect_L7.2mm_W7.2mm_P5.00mm_FKS2_FKP2_MKS2_MKP2
- C15, C5, C8: footprint Capacitor_THT:C_Rect_L7.0mm_W2.5mm_P5.00mm -> Capacitor_THT:C_Rect_L16.5mm_W11.8mm_P15.00mm_MKT
- RV5: value 4k7 -> 10k
- RV6: value 500k -> 1M
Changed lines of the file:
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@@
 			)
 		)
-		(property "Value" "500k"
+		(property "Value" "1M"
 			(at 140.97 180.34 90)
 			(show_name no)
@@
 			)
 		)
-		(property "Footprint" "Capacitor_THT:C_Rect_L7.0mm_W2.5mm_P5.00mm"
+		(property "Footprint" "Capacitor_THT:C_Rect_L16.5mm_W11.8mm_P15.00mm_MKT"
 			(at 50.8 62.23 0)
 			(hide yes)
@@
 			)
 		)
-		(property "Footprint" "Capacitor_THT:C_Rect_L7.0mm_W2.5mm_P5.00mm"
+		(property "Footprint" "Capacitor_THT:C_Rect_L16.5mm_W7.3mm_P15.00mm_MKT"
 			(at 91.44 52.07 0)
 			(hide yes)
@@
 			)
 		)
-		(property "Footprint" "Capacitor_THT:C_Rect_L7.0mm_W2.5mm_P5.00mm"
+		(property "Footprint" "Capacitor_THT:C_Rect_L16.5mm_W11.8mm_P15.00mm_MKT"
 			(at 44.45 48.26 0)
 			(hide yes)
@@
 			)
 		)
-		(property "Footprint" "Capacitor_THT:C_Rect_L7.0mm_W2.5mm_P5.00mm"
+		(property "Footprint" "Capacitor_THT:C_Rect_L16.5mm_W7.3mm_P15.00mm_MKT"
 			(at 96.52 80.01 0)
 			(hide yes)
@@
 			)
 		)
-		(property "Footprint" "Capacitor_THT:C_Rect_L7.0mm_W2.5mm_P5.00mm"
+		(property "Footprint" "Capacitor_THT:C_Rect_L7.2mm_W7.2mm_P5.00mm_FKS2_FKP2_MKS2_MKP2"
 			(at 340.36 138.43 0)
 			(hide yes)
@@
 			)
 		)
-		(property "Footprint" "Capacitor_THT:C_Rect_L7.0mm_W2.5mm_P5.00mm"
+		(property "Footprint" "Capacitor_THT:C_Rect_L16.5mm_W11.8mm_P15.00mm_MKT"
 			(at 128.27 186.69 0)
 			(hide yes)
@@
 			)
 		)
-		(property "Value" "4k7"
+		(property "Value" "10k"
 			(at 98.552 180.34 90)
 			(show_name no)
@@
 			)
 		)
-		(property "Footprint" "Capacitor_THT:C_Rect_L7.0mm_W2.5mm_P5.00mm"
+		(property "Footprint" "Capacitor_THT:C_Rect_L7.2mm_W7.2mm_P5.00mm_FKS2_FKP2_MKS2_MKP2"
 			(at 57.15 128.27 0)
 			(hide yes)
