File: kicad_withpcb/compressor_front/compressor_front.kicad_pcb (KiCad board)
At the start: 2 copper layers, 35 x 110 mm, 33 parts, among them J1 MAIN BOARD, SW1 BYPASS, SW2 INT/EXT, SW3 HPF DEFEAT, SW4 LINK, U10 LM3915, U9 LM3914

Commit message: Use the Jaycar sub-miniature toggles on the front board
Footprints for the ST0300 (SPDT) from its datasheet: solder lugs on
2.54 mm in slotted holes, 8.13 x 5.08 mm body. The ST0310 (DPDT) has no
published drawing, so its footprint assumes the same pitch with rows
4.7 mm apart. The board now sits about 8.7 mm behind the panel with the
switch bodies resting on it. Re-routed.

DRC: 0 errors, 0 unconnected, schematic parity clean.

Co-Authored-By: Claude Opus 5.5 (1M context) <noreply@anthropic.com>
Parts:
- SW1: footprint compressor_front:SW_Toggle_Mini_DPDT -> compressor_front:SW_Toggle_SubMini_DPDT_Jaycar_ST0310
- SW2, SW3, SW4: footprint compressor_front:SW_Toggle_Mini_SPDT -> compressor_front:SW_Toggle_SubMini_SPDT_Jaycar_ST0300
Routing:
- net LVL_METER: track 142.5 -> 109.0 mm, vias 1 -> 0
- net +16V: track 216.1 -> 203.1 mm
- net BYP_B: track 36.9 -> 25.0 mm, vias 2 -> 0
- net OUT-A: track 37.1 -> 48.0 mm
- net MAKEUP_FB: track 36.2 -> 46.0 mm
- net GR_REF: track 136.3 -> 126.7 mm, vias 0 -> 1
- net GR_METER: track 113.4 -> 104.8 mm
- net SIG-VCA: track 60.8 -> 53.1 mm, vias 1 -> 0
- net HPF_B: track 64.9 -> 71.5 mm, vias 0 -> 1
- net KEY_SRC: track 56.6 -> 50.8 mm, vias 2 -> 0
- net OUT+: track 23.4 -> 18.2 mm
- net RATIO_CW: track 40.4 -> 35.3 mm, vias 1 -> 0
- net LINK: track 45.3 -> 50.3 mm, vias 0 -> 1
- net KEY: track 48.1 -> 51.5 mm
- net AGND: track 191.8 -> 189.2 mm, vias 1 -> 0
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Other:
- board text added: "Front of board faces the panel, about 8.7 mm behind it: the toggle bodies rest on the board."
- board text added: "Panel 38.10 x 133.35, origin top-left. Holes: pots 7.2, toggles 5.2, LEDs 2.2"
- board text removed: "Front of board faces the panel. Board sits 10 mm behind it."
- board text removed: "Panel 38.10 x 133.35, origin top-left. Holes: pots 7.2, toggles 6.5, LEDs 2.2"

Commit message: Add 3D models for the pots and toggles
KiCad ships no model for the Alps RK09K or the Jaycar sub-miniature
toggles, so the front board showed bare footprints in 3D and in STEP.

- Pots: Alps' own RK09K1130 STEP, fetched by tools/get_3d_models.sh rather
  than committed, on a project copy of the stock footprint that places it
  on the shaft centre
- Toggles: simple solids to the ST0300 datasheet, generated by
  tools/make_toggle_models.py

Every other part already had a library model. STEP export of both boards
now includes every component.

Co-Authored-By: Claude Opus 5.5 (1M context) <noreply@anthropic.com>
Parts:
- RV2, RV3, RV4, RV5, RV6: footprint Potentiometer_THT:Potentiometer_Alps_RK09K_Single_Vertical -> compressor_front:Potentiometer_Alps_RK09K_Single_Vertical
Changed lines of the file:
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@@
 		)
 		(embedded_fonts no)
+		(model "${KIPRJMOD}/3dmodels/SW_Toggle_SubMini_DPDT_Jaycar_ST0310.step"
+			(offset
+				(xyz 0 0 0)
+			)
+			(scale
+				(xyz 1 1 1)
+			)
+			(rotate
+				(xyz 0 0 0)
+			)
+		)
 	)
 	(footprint "LED_THT:LED_D2.0mm_W4.0mm_H2.8mm_FlatTop"
@@
 		)
 	)
-	(footprint "Potentiometer_THT:Potentiometer_Alps_RK09K_Single_Vertical"
+	(footprint "compressor_front:Potentiometer_Alps_RK09K_Single_Vertical"
 		(layer "F.Cu")
 		(at 116.55 120 90)
@@
 		)
 		(embedded_fonts no)
-		(model "${KICAD10_3DMODEL_DIR}/Potentiometer_THT.3dshapes/Potentiometer_Alps_RK09K_Single_Vertical.step"
+		(model "${KIPRJMOD}/3dmodels/RK09K1130-20.STEP"
 			(offset
-				(xyz 0 0 0)
+				(xyz 7.5 -2.5 6)
 			)
 			(scale
@@
 			)
 			(rotate
-				(xyz 0 0 0)
+				(xyz 0 0 90)
 			)
 		)
@@
 		)
 	)
-	(footprint "Potentiometer_THT:Potentiometer_Alps_RK09K_Single_Vertical"
+	(footprint "compressor_front:Potentiometer_Alps_RK09K_Single_Vertical"
 		(layer "F.Cu")
 		(at 122.6 138.5 90)
@@
 		)
 		(embedded_fonts no)
-		(model "${KICAD10_3DMODEL_DIR}/Potentiometer_THT.3dshapes/Potentiometer_Alps_RK09K_Single_Vertical.step"
+		(model "${KIPRJMOD}/3dmodels/RK09K1130-20.STEP"
 			(offset
-				(xyz 0 0 0)
+				(xyz 7.5 -2.5 6)
 			)
 			(scale
@@
 			)
 			(rotate
-				(xyz 0 0 0)
+				(xyz 0 0 90)
 			)
 		)
 	)
-	(footprint "Potentiometer_THT:Potentiometer_Alps_RK09K_Single_Vertical"
+	(footprint "compressor_front:Potentiometer_Alps_RK09K_Single_Vertical"
 		(layer "F.Cu")
 		(at 116.55 99.5 90)
@@
 		)
 		(embedded_fonts no)
-		(model "${KICAD10_3DMODEL_DIR}/Potentiometer_THT.3dshapes/Potentiometer_Alps_RK09K_Single_Vertical.step"
+		(model "${KIPRJMOD}/3dmodels/RK09K1130-20.STEP"
 			(offset
-				(xyz 0 0 0)
+				(xyz 7.5 -2.5 6)
 			)
 			(scale
@@
 			)
 			(rotate
-				(xyz 0 0 0)
+				(xyz 0 0 90)
 			)
 		)
@@
 		)
 	)
-	(footprint "Potentiometer_THT:Potentiometer_Alps_RK09K_Single_Vertical"
+	(footprint "compressor_front:Potentiometer_Alps_RK09K_Single_Vertical"
 		(layer "F.Cu")
 		(at 107.5 138.5 90)
@@
 		)
 		(embedded_fonts no)
-		(model "${KICAD10_3DMODEL_DIR}/Potentiometer_THT.3dshapes/Potentiometer_Alps_RK09K_Single_Vertical.step"
+		(model "${KIPRJMOD}/3dmodels/RK09K1130-20.STEP"
 			(offset
-				(xyz 0 0 0)
+				(xyz 7.5 -2.5 6)
 			)
 			(scale
@@
 			)
 			(rotate
-				(xyz 0 0 0)
+				(xyz 0 0 90)
 			)
 		)
@@
 		)
 		(embedded_fonts no)
+		(model "${KIPRJMOD}/3dmodels/SW_Toggle_SubMini_SPDT_Jaycar_ST0300.step"
+			(offset
+				(xyz 0 0 0)
+			)
+			(scale
+				(xyz 1 1 1)
+			)
+			(rotate
+				(xyz 0 0 0)
+			)
+		)
 	)
 	(footprint "compressor_front:SW_Toggle_SubMini_SPDT_Jaycar_ST0300"
@@
 		)
 		(embedded_fonts no)
+		(model "${KIPRJMOD}/3dmodels/SW_Toggle_SubMini_SPDT_Jaycar_ST0300.step"
+			(offset
+				(xyz 0 0 0)
+			)
+			(scale
+				(xyz 1 1 1)
+			)
+			(rotate
+				(xyz 0 0 0)
+			)
+		)
 	)
-	(footprint "Potentiometer_THT:Potentiometer_Alps_RK09K_Single_Vertical"
+	(footprint "compressor_front:Potentiometer_Alps_RK09K_Single_Vertical"
 		(layer "F.Cu")
 		(at 116.55 158.5 90)
@@
 		)
 		(embedded_fonts no)
-		(model "${KICAD10_3DMODEL_DIR}/Potentiometer_THT.3dshapes/Potentiometer_Alps_RK09K_Single_Vertical.step"
+		(model "${KIPRJMOD}/3dmodels/RK09K1130-20.STEP"
 			(offset
-				(xyz 0 0 0)
+				(xyz 7.5 -2.5 6)
 			)
 			(scale
@@
 			)
 			(rotate
-				(xyz 0 0 0)
+				(xyz 0 0 90)
 			)
 		)
@@
 		)
 		(embedded_fonts no)
+		(model "${KIPRJMOD}/3dmodels/SW_Toggle_SubMini_SPDT_Jaycar_ST0300.step"
+			(offset
+				(xyz 0 0 0)
+			)
+			(scale
+				(xyz 1 1 1)
+			)
+			(rotate
+				(xyz 0 0 0)
+			)
+		)
 	)
 	(footprint "Connector_PinHeader_2.54mm:PinHeader_2x15_P2.54mm_Vertical"
