File: kicad_withpcb/compressor_front/compressor_front.kicad_sch (KiCad schematic)
At the start: 33 parts, among them J1 MAIN BOARD, SW1 BYPASS, SW2 INT/EXT, SW3 HPF DEFEAT, SW4 LINK, U10 LM3915, U9 LM3914

Commit message: Use the Jaycar sub-miniature toggles on the front board
Footprints for the ST0300 (SPDT) from its datasheet: solder lugs on
2.54 mm in slotted holes, 8.13 x 5.08 mm body. The ST0310 (DPDT) has no
published drawing, so its footprint assumes the same pitch with rows
4.7 mm apart. The board now sits about 8.7 mm behind the panel with the
switch bodies resting on it. Re-routed.

DRC: 0 errors, 0 unconnected, schematic parity clean.

Co-Authored-By: Claude Opus 5.5 (1M context) <noreply@anthropic.com>
Parts:
- SW1: footprint compressor_front:SW_Toggle_Mini_DPDT -> compressor_front:SW_Toggle_SubMini_DPDT_Jaycar_ST0310
- SW2, SW3, SW4: footprint compressor_front:SW_Toggle_Mini_SPDT -> compressor_front:SW_Toggle_SubMini_SPDT_Jaycar_ST0300
Changed lines of the file:
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@@
 			)
 		)
-		(property "Footprint" "compressor_front:SW_Toggle_Mini_SPDT"
+		(property "Footprint" "compressor_front:SW_Toggle_SubMini_SPDT_Jaycar_ST0300"
 			(at 277.622 104.14 0)
 			(hide yes)
@@
 			)
 		)
-		(property "Footprint" "compressor_front:SW_Toggle_Mini_SPDT"
+		(property "Footprint" "compressor_front:SW_Toggle_SubMini_SPDT_Jaycar_ST0300"
 			(at 229.87 95.25 0)
 			(hide yes)
@@
 			)
 		)
-		(property "Footprint" "compressor_front:SW_Toggle_Mini_SPDT"
+		(property "Footprint" "compressor_front:SW_Toggle_SubMini_SPDT_Jaycar_ST0300"
 			(at 190.5 95.25 0)
 			(hide yes)
@@
 			)
 		)
-		(property "Footprint" "compressor_front:SW_Toggle_Mini_DPDT"
+		(property "Footprint" "compressor_front:SW_Toggle_SubMini_DPDT_Jaycar_ST0310"
 			(at 110.49 95.25 0)
 			(hide yes)
@@
 			)
 		)
-		(property "Footprint" "compressor_front:SW_Toggle_Mini_DPDT"
+		(property "Footprint" "compressor_front:SW_Toggle_SubMini_DPDT_Jaycar_ST0310"
 			(at 149.86 95.25 0)
 			(hide yes)

Commit message: Add 3D models for the pots and toggles
KiCad ships no model for the Alps RK09K or the Jaycar sub-miniature
toggles, so the front board showed bare footprints in 3D and in STEP.

- Pots: Alps' own RK09K1130 STEP, fetched by tools/get_3d_models.sh rather
  than committed, on a project copy of the stock footprint that places it
  on the shaft centre
- Toggles: simple solids to the ST0300 datasheet, generated by
  tools/make_toggle_models.py

Every other part already had a library model. STEP export of both boards
now includes every component.

Co-Authored-By: Claude Opus 5.5 (1M context) <noreply@anthropic.com>
Parts:
- RV2, RV3, RV4, RV5, RV6: footprint Potentiometer_THT:Potentiometer_Alps_RK09K_Single_Vertical -> compressor_front:Potentiometer_Alps_RK09K_Single_Vertical
Changed lines of the file:
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@@
 			)
 		)
-		(property "Footprint" "Potentiometer_THT:Potentiometer_Alps_RK09K_Single_Vertical"
+		(property "Footprint" "compressor_front:Potentiometer_Alps_RK09K_Single_Vertical"
 			(at 270.51 49.53 0)
 			(hide yes)
@@
 			)
 		)
-		(property "Footprint" "Potentiometer_THT:Potentiometer_Alps_RK09K_Single_Vertical"
+		(property "Footprint" "compressor_front:Potentiometer_Alps_RK09K_Single_Vertical"
 			(at 190.5 49.53 0)
 			(hide yes)
@@
 			)
 		)
-		(property "Footprint" "Potentiometer_THT:Potentiometer_Alps_RK09K_Single_Vertical"
+		(property "Footprint" "compressor_front:Potentiometer_Alps_RK09K_Single_Vertical"
 			(at 110.49 49.53 0)
 			(hide yes)
@@
 			)
 		)
-		(property "Footprint" "Potentiometer_THT:Potentiometer_Alps_RK09K_Single_Vertical"
+		(property "Footprint" "compressor_front:Potentiometer_Alps_RK09K_Single_Vertical"
 			(at 229.87 49.53 0)
 			(hide yes)
@@
 			)
 		)
-		(property "Footprint" "Potentiometer_THT:Potentiometer_Alps_RK09K_Single_Vertical"
+		(property "Footprint" "compressor_front:Potentiometer_Alps_RK09K_Single_Vertical"
 			(at 149.86 49.53 0)
 			(hide yes)
