File: kicad/power.kicad_sch (KiCad schematic)
At the start: 47 parts, among them U1 NE5532, U2 NE5532, U3 NE5532, U4 TL072, U5 NE5532, U6 NE5532, U7 NE5532

Commit message: Bring the compressor's values in line with the design targets
Through gain: R21/R22 3k3 to 6k8 halves the recovery amp's gain, so the
module is unity balanced in to out and BYPASS matches; R36 100k to 200k
keeps the detector's level. Bass: C9/C10 2u2 to 4u7 with the larger
input resistors puts the -3 dB point near 5 Hz.
Threshold: RV3 1M linear to 250k audio taper and R35 20k to 2k4 spread
about -20 to +20 dBu over the knob. R60 47k to 24k sets the resting
steer near 150 mV.
Timing: R45/R46/RV5 and R47/RV6/R74 scaled up to match the RC targets
with the same C15.

Same changes on the sheets, both boards and design.py. The simulation's
pot model gains an audio taper, and the burst test now runs at half
threshold.
Parts:
- R60: value 47k -> 24k
Changed lines of the file:
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@@
 			)
 		)
-		(property "Value" "47k"
+		(property "Value" "24k"
 			(at 64.77 109.728 90)
 			(show_name no)

Commit message: Stop the fast-attack overshoot: C22 47u to 4u7
C22 made STA lag STB by about 60 ms, so when CTRL-B pulled the
reference node down the steering kept moving after the control
voltage had settled, overshooting by up to 20 dB. With 4u7 the two
sides track and the overshoot is about 1 dB. RV5 back to 4k7 and RV6
to 500k, since the attack and release run slower without it.
Parts:
- C22: value 47u -> 4u7
Changed lines of the file:
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@@
 			)
 		)
-		(property "Value" "47u"
+		(property "Value" "4u7"
 			(at 92.964 112.268 90)
 			(show_name no)
