File: kicad/sidechain.kicad_sch (KiCad schematic)
At the start: 30 parts, among them SW2 INT/EXT, SW3 HPF DEFEAT, SW4 LINK, U3 NE5532, U4 TL072, U6 NE5532

Commit message: Simulate the compressor, fix its values, and fit Altronics parts (#5)
* Make the schematic simulate in KiCad, and add the simulation results

Every part on the kicad/ sheets now has a SPICE model (Sim.* fields, models in
kicad/sim/compressor_models.lib), the connectors are excluded from simulation, and the
root sheet carries a test bench: the rack's supplies, a balanced source, a load and the
knob settings as .param lines. The netlist is unchanged.

tools/add_sim_models.py writes the fields. tools/sim/run_all.py exports the netlist with
kicad-cli and runs the characterisation in ngspice; kicad/sim/README.md has how to run
it in KiCad and what it found.

* Bring the compressor's values in line with the design targets

Through gain: R21/R22 3k3 to 6k8 halves the recovery amp's gain, so the
module is unity balanced in to out and BYPASS matches; R36 100k to 200k
keeps the detector's level. Bass: C9/C10 2u2 to 4u7 with the larger
input resistors puts the -3 dB point near 5 Hz.
Threshold: RV3 1M linear to 250k audio taper and R35 20k to 2k4 spread
about -20 to +20 dBu over the knob. R60 47k to 24k sets the resting
steer near 150 mV.
Timing: R45/R46/RV5 and R47/RV6/R74 scaled up to match the RC targets
with the same C15.

Same changes on the sheets, both boards and design.py. The simulation's
pot model gains an audio taper, and the burst test now runs at half
threshold.

* Carry the new values onto both boards' schematics and layouts

* Retune attack and release: R45 220R, R46 47R, RV5 10k, R47 15k

The first pass ran the attack too slow (9 to 103 ms against a 2.7 to
50 ms target). Results are regenerated in the next commit.

* Regenerate the simulation results for the new values

* Stop the fast-attack overshoot: C22 47u to 4u7

C22 made STA lag STB by about 60 ms, so when CTRL-B pulled the
reference node down the steering kept moving after the control
voltage had settled, overshooting by up to 20 dB. With 4u7 the two
sides track and the overshoot is about 1 dB. RV5 back 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
Parts:
- C14: value 220n -> 2u2; footprint Capacitor_THT:C_Rect_L7.0mm_W2.5mm_P5.00mm -> Capacitor_THT:C_Rect_L7.2mm_W7.2mm_P5.00mm_FKS2_FKP2_MKS2_MKP2
- C15: footprint Capacitor_THT:C_Rect_L7.0mm_W2.5mm_P5.00mm -> Capacitor_THT:C_Rect_L16.5mm_W11.8mm_P15.00mm_MKT
- R35: value 20k -> 1k
- R36: value 100k -> 82k
- R38: value 10k -> 1k
- R47: value 4k7 -> 15k
- RV3: value 1M -> 100kA
- RV5: value 4k7 -> 10k
- RV6: value 220k -> 1M
