File: kicad/sidechain.kicad_sch (KiCad schematic)
At the start: 30 parts, among them SW2 INT/EXT, SW3 HPF DEFEAT, SW4 LINK, U3 NE5532, U4 TL072, U6 NE5532

Commit message: Use 100k pots for RV3 and RV6, and steady the sidechain high-pass
RK09K pots stop at 100k. RV3 becomes 100kA with R35 1k and R36 82k,
which scales the threshold network and keeps the -20 to +20 dBu range.
RV6 becomes 100k, so the slowest release drops to about 0.4 s.

R35 at 2k4 had also loaded the sidechain high-pass (C14 into R38), so at
the lowest threshold its corner rose to about 400 Hz. R38 1k and C14 2u2
hold it between about 80 and 160 Hz across the threshold knob.
Parts:
- C14: value 220n -> 2u2
- R35: value 2k4 -> 1k
- R36: value 200k -> 82k
- R38: value 10k -> 1k
- RV3: value 250kA -> 100kA
- RV6: value 500k -> 100k
Changed lines of the file:
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@@
 			)
 		)
-		(property "Value" "220n"
+		(property "Value" "2u2"
 			(at 156.21 67.31 90)
 			(show_name no)
@@
 			)
 		)
-		(property "Value" "10k"
+		(property "Value" "1k"
 			(at 167.386 74.168 90)
 			(show_name no)
@@
 			)
 		)
-		(property "Value" "2k4"
+		(property "Value" "1k"
 			(at 187.96 65.786 90)
 			(show_name no)
@@
 			)
 		)
-		(property "Value" "250kA"
+		(property "Value" "100kA"
 			(at 175.006 60.452 90)
 			(show_name no)
@@
 			)
 		)
-		(property "Sim.Params" "R=250000 POS={THRESHOLD} TAPER=1"
+		(property "Sim.Params" "R=100000 POS={THRESHOLD} TAPER=1"
 			(at 172.72 63.5 90)
 			(show_name no)
@@
 			)
 		)
-		(property "Value" "500k"
+		(property "Value" "100k"
 			(at 243.84 118.11 90)
 			(show_name no)
@@
 			)
 		)
-		(property "Sim.Params" "R=500000 POS={RELEASE}"
+		(property "Sim.Params" "R=100000 POS={RELEASE}"
 			(at 238.76 116.84 90)
 			(show_name no)
@@
 			)
 		)
-		(property "Value" "200k"
+		(property "Value" "82k"
 			(at 211.074 68.58 90)
 			(show_name no)

Commit message: Put RV6 back to 500k, to be a Bourns PTV09
RK09K stops at 100k, which would cut the slowest release to about 0.4 s.
Lyn chose a 500k Bourns PTV09 instead, keeping it near 1.8 s.
Parts:
- RV6: value 100k -> 500k
Changed lines of the file:
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@@
 			)
 		)
-		(property "Value" "100k"
+		(property "Value" "500k"
 			(at 243.84 118.11 90)
 			(show_name no)
@@
 			)
 		)
-		(property "Sim.Params" "R=100000 POS={RELEASE}"
+		(property "Sim.Params" "R=500000 POS={RELEASE}"
 			(at 238.76 116.84 90)
 			(show_name no)

Commit message: Fit real film capacitors on the main board and use Altronics pots for RV5/RV6
RV5 (ATTACK) goes 4k7 -> 10k and RV6 (RELEASE) 500k -> 1M, the nearest
Altronics 9 mm values (R1946, R1950), on the split sheets, both boards
and design.py; the Sim.Params follow (R=10000, R=1e+06).

C5, C8, C9, C10, C14, C15 and C35 were drawn as 7 x 2.5 mm on 5 mm, which
no 2.2-10 uF film part fits. They now use stock KiCad footprints for
in-stock element14 parts:
  10 uF  C5 C8 C15  TDK B32562H1106K000   C_Rect_L16.5mm_W11.8mm_P15.00mm_MKT
  4.7 uF C9 C10     TDK B32562H1475K000   C_Rect_L16.5mm_W7.3mm_P15.00mm_MKT
  2.2 uF C14 C35    KEMET MMK5225K63J06L4 C_Rect_L7.2mm_W7.2mm_P5.00mm_FKS2...

To make room, small parts were re-placed by script (the caps near their
old spots, displaced parts re-homed, then same-footprint parts swapped to
cut wire length; transistors, ICs, connectors and trimmers did not move)
and the main board was re-routed with Freerouting, keeping the original
card-finger stubs. DRC 0 errors, 0 unconnected, schematic parity clean;
ERC 0 errors. The BOM names the element14 parts.
Parts:
- C14: footprint Capacitor_THT:C_Rect_L7.0mm_W2.5mm_P5.00mm -> Capacitor_THT:C_Rect_L7.2mm_W7.2mm_P5.00mm_FKS2_FKP2_MKS2_MKP2
- C15: footprint Capacitor_THT:C_Rect_L7.0mm_W2.5mm_P5.00mm -> Capacitor_THT:C_Rect_L16.5mm_W11.8mm_P15.00mm_MKT
- RV5: value 4k7 -> 10k
- RV6: value 500k -> 1M
Changed lines of the file:
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@@
 			)
 		)
-		(property "Footprint" "Capacitor_THT:C_Rect_L7.0mm_W2.5mm_P5.00mm"
+		(property "Footprint" "Capacitor_THT:C_Rect_L7.2mm_W7.2mm_P5.00mm_FKS2_FKP2_MKS2_MKP2"
 			(at 160.02 66.04 0)
 			(hide yes)
@@
 			)
 		)
-		(property "Value" "4k7"
+		(property "Value" "10k"
 			(at 201.422 118.11 90)
 			(show_name no)
@@
 			)
 		)
-		(property "Sim.Params" "R=4700 POS={ATTACK}"
+		(property "Sim.Params" "R=10000 POS={ATTACK}"
 			(at 196.85 116.84 90)
 			(show_name no)
@@
 			)
 		)
-		(property "Footprint" "Capacitor_THT:C_Rect_L7.0mm_W2.5mm_P5.00mm"
+		(property "Footprint" "Capacitor_THT:C_Rect_L16.5mm_W11.8mm_P15.00mm_MKT"
 			(at 231.14 124.46 0)
 			(hide yes)
@@
 			)
 		)
-		(property "Value" "500k"
+		(property "Value" "1M"
 			(at 243.84 118.11 90)
 			(show_name no)
@@
 			)
 		)
-		(property "Sim.Params" "R=500000 POS={RELEASE}"
+		(property "Sim.Params" "R=1e+06 POS={RELEASE}"
 			(at 238.76 116.84 90)
 			(show_name no)

Commit message: Re-route the main board, reverse RATIO, and re-plot the Gerbers for both boards (#7)
* Re-plot the Gerbers for both boards from the current layout

The committed main-board Gerbers were plotted on 2026-10-01, before the film-cap
re-place and re-route, so 119 of their holes no longer match the board. Re-plot
them from the current board, add the front board's set, and zip each for the fab.

tools/plot_fab.sh does both boards in one go so the zips can be refreshed after
every board change. The README gets an Ordering section with the fab settings.

* Re-route the main board: paired IN/OUT, one-piece ground pour

IN+/IN- and OUT+/OUT- run as pairs 0.6 mm apart on the top layer, with
one via each on IN- and OUT- beside the edge fingers. Most other tracks
moved to the top so the bottom AGND pour is one piece (was seven).
DRC 0 errors, 0 unconnected, 0 schematic parity issues. Gerbers re-plotted.

* Swap RATIO's outer pins so clockwise gives a harder ratio

RV4 pin 1 is now AGND and pin 3 RATIO_CW on all three schematics and the
front board (symbol mirrored, front-board tracks re-routed at RV4).
The sim model reads POS={1-RATIO}, so RATIO keeps its meaning and the
results are unchanged. Front-board DRC 0 errors, 0 unconnected, 0 parity;
front Gerbers re-plotted.
Connections:
- net AGND: now also RV4.1; no longer RV4.3
- net RATIO_CW: now also RV4.3; no longer RV4.1
Changed lines of the file:
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@@
 		(lib_id "Device:R_Potentiometer")
 		(at 166.37 123.19 0)
+		(mirror x)
 		(unit 1)
 		(body_style 1)
@@
 			)
 		)
-		(property "Sim.Params" "R=100000 POS={RATIO}"
+		(property "Sim.Params" "R=100000 POS={1-RATIO}"
 			(at 166.37 123.19 0)
 			(show_name no)
