File: kicad/meters.kicad_sch (KiCad schematic)
At the start: 36 parts, among them U10 LM3915, U7 NE5532, U9 LM3914

Commit message: Two LM3914 meters with ten LEDs each, simulated (#6)
* Swap the level meter's LM3915 for an LM3914 on outputs 1-7

Nobody stocks the LM3915, so U10 becomes a second LM3914. The LEDs move
to outputs 1-7 and outputs 8-10 join the top LED, giving a 17 dB scale
with no added parts. Front board LVL tracks re-routed; BOM regenerated.

* Give both meters ten LEDs and simulate them

Adds D27-D29 (GR outputs 8-10) and D37-D39 (LVL outputs 8-10) on all three
schematics. The front board's meter columns move to a 3.0 mm pitch with
LVL output 10 at the top; R90/R92 move to a 7.62 mm footprint and C38
turns to clear the LEDs; the affected nets were re-routed. R92 becomes 4k7
so RV8 can set the top LED at +18 dBu. The panel gets the six extra holes.
The LM3914 sim model now has its comparators and LED current sinks, and
tools/sim/meters.py simulates both meters.

* Write up the meter simulation
Parts:
- added D27, D28, D29, D37, D38, D39: meter, LED_THT:LED_D2.0mm_W4.0mm_H2.8mm_FlatTop, symbol Device:LED
- R90: footprint Resistor_THT:R_Axial_DIN0207_L6.3mm_D2.5mm_P10.16mm_Horizontal -> Resistor_THT:R_Axial_DIN0207_L6.3mm_D2.5mm_P7.62mm_Horizontal
- R92: value 8k2 -> 4k7; footprint Resistor_THT:R_Axial_DIN0207_L6.3mm_D2.5mm_P10.16mm_Horizontal -> Resistor_THT:R_Axial_DIN0207_L6.3mm_D2.5mm_P7.62mm_Horizontal
- U10: value LM3915 -> LM3914
Connections:
- net +16V: now also D27.2 (A), D28.2 (A), D29.2 (A), D37.2 (A), D38.2 (A), D39.2 (A)
- net LVLL6: now reaches D35.1 (K)
- net LVLL6: now also U10.14 (LED6); no longer U10.11 (LED9)
- net LVLL1: now reaches D30.1 (K)
- net LVLL1: now also U10.1 (LED1); no longer U10.16 (LED4)
- net LVLL10: now reaches U10.10 (LED10)
- net LVLL10: now also D39.1 (K); no longer D36.1 (K)
- net LVLL5: now reaches D34.1 (K)
- net LVLL5: now also U10.15 (LED5); no longer U10.12 (LED8)
- net LVLL4: now reaches D33.1 (K)
- net LVLL4: now also U10.16 (LED4); no longer U10.13 (LED7)
- net LVLL3: now reaches D32.1 (K)
- net LVLL3: now also U10.17 (LED3); no longer U10.14 (LED6)
- net LVLL2: now reaches D31.1 (K)
- net LVLL2: now also U10.18 (LED2); no longer U10.15 (LED5)
- net GRL10: now reaches U9.10 (LED10)
- net GRL10: now also D29.1 (K)
- net GRL9: now reaches U9.11 (LED9)
- net GRL9: now also D28.1 (K)
- net GRL8: now reaches U9.12 (LED8)
- net GRL8: now also D27.1 (K)
- new net LVLL7: D36.1 (K), U10.13 (LED7)
- new net LVLL8: D37.1 (K), U10.12 (LED8)
- new net LVLL9: D38.1 (K), U10.11 (LED9)
- no-connect marks 8 -> 2
